Commit message: update axol joint limits

File: almond_axol/kinematics/urdf/axol.urdf (robot description, URDF)
Before this commit: robot assembly, 18 links, 17 joints
Joints:
- joint left_e1_0: limit (none) -> lower=0.0 upper=2.6389 effort=87.0 velocity=30.0; type continuous -> revolute
- joint left_e2_0: limit (none) -> lower=-1.5708 upper=1.5708 effort=87.0 velocity=30.0; type continuous -> revolute
- joint left_s1_0: limit (none) -> lower=-1.5708 upper=1.5708 effort=87.0 velocity=30.0; type continuous -> revolute
- joint left_s2_0: limit (none) -> lower=-1.5708 upper=0.1885 effort=87.0 velocity=30.0; type continuous -> revolute
- joint left_s3_0: limit (none) -> lower=-1.5708 upper=1.5708 effort=87.0 velocity=30.0; type continuous -> revolute
- joint left_w1_0: limit (none) -> lower=-1.5708 upper=1.5708 effort=87.0 velocity=30.0; type continuous -> revolute
- joint left_w2_0: limit (none) -> lower=-1.5708 upper=1.5708 effort=87.0 velocity=30.0; type continuous -> revolute
- joint right_e1_0: limit (none) -> lower=0.0 upper=2.6389 effort=87.0 velocity=30.0; type continuous -> revolute
- joint right_e2_0: limit (none) -> lower=-1.5708 upper=1.5708 effort=87.0 velocity=30.0; type continuous -> revolute
- joint right_s1_0: limit (none) -> lower=-1.5708 upper=1.5708 effort=87.0 velocity=30.0; type continuous -> revolute
- joint right_s2_0: limit (none) -> lower=-0.1885 upper=1.5708 effort=87.0 velocity=30.0; type continuous -> revolute
- joint right_s3_0: limit (none) -> lower=-1.5708 upper=1.5708 effort=87.0 velocity=30.0; type continuous -> revolute
- joint right_w1_0: limit (none) -> lower=-1.5708 upper=1.5708 effort=87.0 velocity=30.0; type continuous -> revolute
- joint right_w2_0: limit (none) -> lower=-1.5708 upper=1.5708 effort=87.0 velocity=30.0; type continuous -> revolute

Commit message: fix part of rest pose for teleop

File: almond_axol/kinematics/urdf/axol.urdf (robot description, URDF)
Before this commit: robot assembly, 18 links, 17 joints
Links:
- link left_e1: geometry visual mesh filename=package://urdf/meshes/Left_E1.stl scale=1 1 1
- link left_e2: geometry visual mesh filename=package://urdf/meshes/Left_E2.stl scale=1 1 1
- link left_gripper: geometry visual mesh filename=package://urdf/meshes/Left Gripper.stl scale=1 1 1
- link left_s2: geometry visual mesh filename=package://urdf/meshes/Left_S2.stl scale=1 1 1
- link left_s3: geometry visual mesh filename=package://urdf/meshes/Left_S3.stl scale=1 1 1
- link left_w0: geometry visual mesh filename=package://urdf/meshes/Left_W0.stl scale=1 1 1
- link left_w1: geometry visual mesh filename=package://urdf/meshes/Left_W1.stl scale=1 1 1
- link left_w2: geometry visual mesh filename=package://urdf/meshes/Left_W2.stl scale=1 1 1
- link right_e1: geometry visual mesh filename=package://urdf/meshes/Right_E1.stl scale=1 1 1
- link right_e2: geometry visual mesh filename=package://urdf/meshes/Right_E2.stl scale=1 1 1
- link right_gripper: geometry visual mesh filename=package://urdf/meshes/Right Gripper.stl scale=1 1 1
- link right_s2: geometry visual mesh filename=package://urdf/meshes/Right_S2.stl scale=1 1 1
- link right_s3: geometry visual mesh filename=package://urdf/meshes/Right_S3.stl scale=1 1 1
- link right_w0: geometry visual mesh filename=package://urdf/meshes/Right_W0.stl scale=1 1 1
- link right_w1: geometry visual mesh filename=package://urdf/meshes/Right_W1.stl scale=1 1 1
- link right_w2: geometry visual mesh filename=package://urdf/meshes/Right_W2.stl scale=1 1 1
- link s1: geometry visual mesh filename=package://urdf/meshes/S1.stl scale=1 1 1

Commit message: fix right elbow joint limit

File: almond_axol/kinematics/urdf/axol.urdf (robot description, URDF)
Before this commit: robot urdf, 18 links, 17 joints
Joints:
- joint right_e1_0: limit lower=0.0 upper=2.6389 effort=87.0 velocity=30.0 -> lower=-2.6389 upper=0.0 effort=87.0 velocity=30.0

Commit message: update urdf

File: almond_axol/kinematics/urdf/axol.urdf (robot description, URDF)
Before this commit: robot urdf, 18 links, 17 joints
Links:
- added link base, mass 0.02496; visual mesh filename=package://assembly/meshes/Base.stl scale=1 1 1
- link left_e1: geometry visual mesh filename=package://assembly/meshes/Left_E1.stl scale=1 1 1
- link left_e2: geometry visual mesh filename=package://assembly/meshes/Left_E2.stl scale=1 1 1
- link left_gripper: geometry visual mesh filename=package://assembly/meshes/Left Gripper.stl scale=1 1 1
- link left_s2: geometry visual mesh filename=package://assembly/meshes/Left_S2.stl scale=1 1 1
- link left_s3: geometry visual mesh filename=package://assembly/meshes/Left_S3.stl scale=1 1 1
- link left_w0: geometry visual mesh filename=package://assembly/meshes/Left_W0.stl scale=1 1 1
- link left_w1: geometry visual mesh filename=package://assembly/meshes/Left_W1.stl scale=1 1 1
- link left_w2: geometry visual mesh filename=package://assembly/meshes/Left_W2.stl scale=1 1 1
- link right_e1: geometry visual mesh filename=package://assembly/meshes/Right_E1.stl scale=1 1 1
- link right_e2: geometry visual mesh filename=package://assembly/meshes/Right_E2.stl scale=1 1 1
- link right_gripper: geometry visual mesh filename=package://assembly/meshes/Right Gripper.stl scale=1 1 1
- link right_s2: geometry visual mesh filename=package://assembly/meshes/Right_S2.stl scale=1 1 1
- link right_s3: geometry visual mesh filename=package://assembly/meshes/Right_S3.stl scale=1 1 1
- link right_w0: geometry visual mesh filename=package://assembly/meshes/Right_W0.stl scale=1 1 1
- link right_w1: geometry visual mesh filename=package://assembly/meshes/Right_W1.stl scale=1 1 1
- link right_w2: geometry visual mesh filename=package://assembly/meshes/Right_W2.stl scale=1 1 1
- link s1: geometry visual mesh filename=package://assembly/meshes/S1.stl scale=1 1 1
Joints:
- added joint base_0: type fixed, parent base, child s1, origin xyz=-2.79001e-17 6.93889e-18 -0.06 rpy=0 -1.06752e-16 0, axis 1.06752e-16 0 1
- joint fixed_node_to_root_joint_0: child s1 -> base; origin xyz=-6.93889e-18 0 0.06 rpy=0 -1.06752e-16 0 -> xyz=-2.77556e-17 -6.93889e-18 0.86 rpy=0 -0 0
- joint left_e1_0: origin xyz=0.04229 2.32031e-17 -0.289385 rpy=-8.89879e-17 3.99879e-31 1.22465e-16 -> xyz=0.04229 1.38514e-17 -0.289385 rpy=-8.89879e-17 3.99879e-31 1.22465e-16
- joint left_e2_0: origin xyz=-0.03229 -1.20261e-17 -0.12429 rpy=1.6148e-14 2.26208e-15 6.65562e-15 -> xyz=-0.03229 -1.38642e-17 -0.12429 rpy=1.6148e-14 2.26208e-15 6.65562e-15
- joint left_gripper_0: origin xyz=0.0285 -1.86926e-17 -0.0335 rpy=0 -0 0 -> xyz=0.0285 -6.93889e-18 -0.0335 rpy=0 -0 0
- joint left_s1_0: origin xyz=0.13 -1.00596e-18 0 rpy=-4.76619e-36 -1.02798e-15 1.03524e-20 -> xyz=0.13 2.46349e-18 0.06 rpy=-4.76619e-36 -1.02798e-15 1.03524e-20
- joint left_s2_0: origin xyz=0.06958 -0.04475 7.14706e-16 rpy=-1.11022e-16 -1.72409e-15 -2.28994e-16 -> xyz=0.06958 -0.04475 4.44089e-16 rpy=-1.11022e-16 -1.72409e-15 -2.28994e-16
- joint left_s3_0: origin xyz=-3.05311e-16 0.04475 -0.07335 rpy=6.12323e-17 -8.04912e-16 -3.52374e-15 -> xyz=-3.88578e-16 0.04475 -0.07335 rpy=6.12323e-17 -8.04912e-16 -3.52374e-15
- joint left_w1_0: origin xyz=0 -0.0285 -0.13567 rpy=1.57652e-14 -1.23165e-16 1.11994e-14 -> xyz=-5.55112e-17 -0.0285 -0.13567 rpy=1.57652e-14 -1.23165e-16 1.11994e-14
- joint right_e1_0: origin xyz=-0.04229 5.0307e-17 -0.289385 rpy=-1.09476e-47 7.39557e-32 1.2326e-32 -> xyz=-0.04229 1.9082e-17 -0.289385 rpy=-1.09476e-47 7.39557e-32 1.2326e-32
- joint right_e2_0: origin xyz=0.03229 -1.04083e-17 -0.12429 rpy=3.03858e-64 4.93038e-32 1.2326e-32 -> xyz=0.03229 -6.93889e-18 -0.12429 rpy=3.03858e-64 4.93038e-32 1.2326e-32
- joint right_gripper_0: origin xyz=-0.0285 1.38778e-17 -0.0335 rpy=3.03858e-64 4.93038e-32 1.2326e-32 -> xyz=-0.0285 -6.93889e-18 -0.0335 rpy=3.03858e-64 4.93038e-32 1.2326e-32
- joint right_s1_0: origin xyz=-0.13 7.27427e-19 -1.38778e-17 rpy=-4.76873e-49 -2.31296e-16 7.65788e-33 -> xyz=-0.13 2.46215e-18 0.06 rpy=-4.76873e-49 -2.31296e-16 7.65788e-33
- joint right_s2_0: origin xyz=-0.06958 -0.04475 3.81639e-16 rpy=-1.28654e-32 -9.17877e-18 -7.824e-17 -> xyz=-0.06958 -0.04475 4.44089e-16 rpy=-1.28654e-32 -9.17877e-18 -7.824e-17

Commit message: fix self collision

File: almond_axol/kinematics/urdf/axol.urdf (robot description, URDF)
Before this commit: robot assembly, 19 links, 18 joints
Links:
- link base: geometry collision mesh filename=package://assembly/meshes/Base.stl scale=1 1 1; visual mesh filename=package://assembly/meshes/Base.stl scale=1 1 1
- link left_e1: geometry collision mesh filename=package://assembly/meshes/Left_E1.stl scale=1 1 1; visual mesh filename=package://assembly/meshes/Left_E1.stl scale=1 1 1
- link left_e2: geometry collision mesh filename=package://assembly/meshes/Left_E2.stl scale=1 1 1; visual mesh filename=package://assembly/meshes/Left_E2.stl scale=1 1 1
- link left_gripper: geometry collision mesh filename=package://assembly/meshes/Left Gripper.stl scale=1 1 1; visual mesh filename=package://assembly/meshes/Left Gripper.stl scale=1 1 1
- link left_s2: geometry collision mesh filename=package://assembly/meshes/Left_S2.stl scale=1 1 1; visual mesh filename=package://assembly/meshes/Left_S2.stl scale=1 1 1
- link left_s3: geometry collision mesh filename=package://assembly/meshes/Left_S3.stl scale=1 1 1; visual mesh filename=package://assembly/meshes/Left_S3.stl scale=1 1 1
- link left_w0: geometry collision mesh filename=package://assembly/meshes/Left_W0.stl scale=1 1 1; visual mesh filename=package://assembly/meshes/Left_W0.stl scale=1 1 1
- link left_w1: geometry collision mesh filename=package://assembly/meshes/Left_W1.stl scale=1 1 1; visual mesh filename=package://assembly/meshes/Left_W1.stl scale=1 1 1
- link left_w2: geometry collision mesh filename=package://assembly/meshes/Left_W2.stl scale=1 1 1; visual mesh filename=package://assembly/meshes/Left_W2.stl scale=1 1 1
- link right_e1: geometry collision mesh filename=package://assembly/meshes/Right_E1.stl scale=1 1 1; visual mesh filename=package://assembly/meshes/Right_E1.stl scale=1 1 1
- link right_e2: geometry collision mesh filename=package://assembly/meshes/Right_E2.stl scale=1 1 1; visual mesh filename=package://assembly/meshes/Right_E2.stl scale=1 1 1
- link right_gripper: geometry collision mesh filename=package://assembly/meshes/Right Gripper.stl scale=1 1 1; visual mesh filename=package://assembly/meshes/Right Gripper.stl scale=1 1 1
- link right_s2: geometry collision mesh filename=package://assembly/meshes/Right_S2.stl scale=1 1 1; visual mesh filename=package://assembly/meshes/Right_S2.stl scale=1 1 1
- link right_s3: geometry collision mesh filename=package://assembly/meshes/Right_S3.stl scale=1 1 1; visual mesh filename=package://assembly/meshes/Right_S3.stl scale=1 1 1
- link right_w0: geometry collision mesh filename=package://assembly/meshes/Right_W0.stl scale=1 1 1; visual mesh filename=package://assembly/meshes/Right_W0.stl scale=1 1 1
- link right_w1: geometry collision mesh filename=package://assembly/meshes/Right_W1.stl scale=1 1 1; visual mesh filename=package://assembly/meshes/Right_W1.stl scale=1 1 1
- link right_w2: geometry collision mesh filename=package://assembly/meshes/Right_W2.stl scale=1 1 1; visual mesh filename=package://assembly/meshes/Right_W2.stl scale=1 1 1
- link s1: geometry collision mesh filename=package://assembly/meshes/S1.stl scale=1 1 1; visual mesh filename=package://assembly/meshes/S1.stl scale=1 1 1

Commit message: fix axol urdf

File: almond_axol/kinematics/urdf/axol.urdf (robot description, URDF)
Before this commit: robot assembly, 19 links, 18 joints
Joints:
- joint left_e1_0: origin xyz=0.04229 1.38514e-17 -0.289385 rpy=-8.89879e-17 3.99879e-31 1.22465e-16 -> xyz=0.04229 1.56381e-16 -0.289385 rpy=1.11022e-16 -4.93529e-16 -6.92805e-17
- joint left_e2_0: origin xyz=-0.03229 -1.38642e-17 -0.12429 rpy=1.6148e-14 2.26208e-15 6.65562e-15 -> xyz=-0.03229 -1.50904e-16 -0.12429 rpy=-8.32667e-17 -6.33174e-17 7.22079e-17
- joint left_gripper_0: origin xyz=0.0285 -6.93889e-18 -0.0335 rpy=0 -0 0 -> xyz=-0.0285 -7.09742e-18 -0.0335 rpy=9.71445e-17 -2.22045e-16 2.77556e-17
- joint left_s1_0: origin xyz=0.13 2.46349e-18 0.06 rpy=-4.76619e-36 -1.02798e-15 1.03524e-20 -> xyz=0.13 9.40122e-18 0.06 rpy=2.77556e-17 -1.02798e-15 1.32751e-21
- joint left_s2_0: origin xyz=0.06958 -0.04475 4.44089e-16 rpy=-1.11022e-16 -1.72409e-15 -2.28994e-16 -> xyz=0.06958 -0.04475 4.44089e-16 rpy=2.498e-16 3.92274e-16 -2.48934e-16
- joint left_s3_0: origin xyz=-3.88578e-16 0.04475 -0.07335 rpy=6.12323e-17 -8.04912e-16 -3.52374e-15 -> xyz=-1.91513e-15 0.04475 -0.07335 rpy=3.33067e-16 -1.05818e-16 -2.03288e-16
- joint left_w1_0: origin xyz=-5.55112e-17 -0.0285 -0.13567 rpy=1.57652e-14 -1.23165e-16 1.11994e-14 -> xyz=-8.32667e-17 -0.0285 -0.13567 rpy=-4.71845e-16 3.45904e-15 -1.18829e-15
- joint left_w2_0: axis 1 0 0 -> -1 0 0; origin xyz=-0.0285 0.0285 -0.057 rpy=-3.36618e-14 -2.11528e-30 -6.12323e-17 -> xyz=0.0285 0.0285 -0.057 rpy=3.4972e-15 -8.32667e-17 -9.70669e-32
- joint right_gripper_0: origin xyz=-0.0285 -6.93889e-18 -0.0335 rpy=3.03858e-64 4.93038e-32 1.2326e-32 -> xyz=0.0285 -6.93889e-18 -0.0335 rpy=-2.71671e-32 1.87354e-29 1.2326e-32
- joint right_w2_0: origin xyz=0.0285 0.0285 -0.057 rpy=3.03858e-64 4.93038e-32 1.2326e-32 -> xyz=0.0285 0.0285 -0.057 rpy=7.5053e-62 -4.93038e-32 -3.14159

Commit message: update urdf

File: almond_axol/kinematics/urdf/axol.urdf (robot description, URDF)
Before this commit: robot assembly, 19 links, 18 joints
Links:
- link left_e2: mass 0.000814328 -> 0.000797087
- link left_w2: mass 4.80988e-05 -> 4.33287e-05
- link right_e2: mass 0.000814328 -> 0.000797087
- link right_w2: mass 4.80988e-05 -> 4.33287e-05
Joints:
- joint left_e2_0: origin xyz=-0.03229 -1.50904e-16 -0.12429 rpy=-8.32667e-17 -6.33174e-17 7.22079e-17 -> xyz=-0.04229 -1.48698e-17 -0.12429 rpy=-8.32667e-17 -6.33174e-17 7.22079e-17
- joint left_gripper_0: origin xyz=-0.0285 -7.09742e-18 -0.0335 rpy=9.71445e-17 -2.22045e-16 2.77556e-17 -> xyz=-0.0285 -7.09742e-18 -0.032251 rpy=9.71445e-17 -2.22045e-16 2.77556e-17
- joint left_w1_0: origin xyz=-8.32667e-17 -0.0285 -0.13567 rpy=-4.71845e-16 3.45904e-15 -1.18829e-15 -> xyz=-5.55112e-17 -0.0285 -0.13567 rpy=-4.71845e-16 3.45904e-15 -1.18829e-15
- joint right_e1_0: origin xyz=-0.04229 1.9082e-17 -0.289385 rpy=-1.09476e-47 7.39557e-32 1.2326e-32 -> xyz=-0.04229 1.47751e-17 -0.289385 rpy=1.07561e-45 7.39557e-32 1.84889e-32
- joint right_e2_0: origin xyz=0.03229 -6.93889e-18 -0.12429 rpy=3.03858e-64 4.93038e-32 1.2326e-32 -> xyz=0.04229 -1.56125e-17 -0.12429 rpy=3.03858e-64 4.93038e-32 1.2326e-32
- joint right_gripper_0: origin xyz=0.0285 -6.93889e-18 -0.0335 rpy=-2.71671e-32 1.87354e-29 1.2326e-32 -> xyz=0.0285 -6.93889e-18 -0.032251 rpy=-2.71671e-32 1.87354e-29 1.2326e-32
- joint right_s3_0: origin xyz=3.88578e-16 0.0323582 -0.07335 rpy=-2.73691e-48 4.93038e-32 4.71657e-48 -> xyz=3.88578e-16 0.04475 -0.07335 rpy=-1.08655e-45 -1.28919e-43 -6.16298e-33

Commit message: a collection of fixes for teleop & can, etc. (#9)
* add option to turn off left or right arm in axol teleop

* add go home sript

* fix disable

* temp fix for wrist3

* tune pid for gripper

* fix gripper

* fix teelop

* fix gripper issue

* fix mit mode

* fix axol urdf

* fix right controller pos

* dont sent myactuator get torque message

* store pos/torque from feedback frames

* update urdf

* can logs and motor bus

* revert bus

* make cameras optional in zed streamer

* create zed test script

* setup ip for zed sender and receiver

* fix pyzed

* improve reader loop

---------

Co-authored-by: Almond Workstation <workstation@almondbot.com>
Co-authored-by: Almond Pi <pi@almond.bot>
Co-authored-by: Almond ZED Box <zed@almond.bot>

File: almond_axol/kinematics/urdf/axol.urdf (robot description, URDF)
Before this commit: robot assembly, 19 links, 18 joints
Links:
- link left_e2: mass 0.000814328 -> 0.000797087
- link left_w2: mass 4.80988e-05 -> 4.33287e-05
- link right_e2: mass 0.000814328 -> 0.000797087
- link right_w2: mass 4.80988e-05 -> 4.33287e-05
Joints:
- joint left_e1_0: origin xyz=0.04229 1.38514e-17 -0.289385 rpy=-8.89879e-17 3.99879e-31 1.22465e-16 -> xyz=0.04229 1.56381e-16 -0.289385 rpy=1.11022e-16 -4.93529e-16 -6.92805e-17
- joint left_e2_0: origin xyz=-0.03229 -1.38642e-17 -0.12429 rpy=1.6148e-14 2.26208e-15 6.65562e-15 -> xyz=-0.04229 -1.48698e-17 -0.12429 rpy=-8.32667e-17 -6.33174e-17 7.22079e-17
- joint left_gripper_0: origin xyz=0.0285 -6.93889e-18 -0.0335 rpy=0 -0 0 -> xyz=-0.0285 -7.09742e-18 -0.032251 rpy=9.71445e-17 -2.22045e-16 2.77556e-17
- joint left_s1_0: origin xyz=0.13 2.46349e-18 0.06 rpy=-4.76619e-36 -1.02798e-15 1.03524e-20 -> xyz=0.13 9.40122e-18 0.06 rpy=2.77556e-17 -1.02798e-15 1.32751e-21
- joint left_s2_0: origin xyz=0.06958 -0.04475 4.44089e-16 rpy=-1.11022e-16 -1.72409e-15 -2.28994e-16 -> xyz=0.06958 -0.04475 4.44089e-16 rpy=2.498e-16 3.92274e-16 -2.48934e-16
- joint left_s3_0: origin xyz=-3.88578e-16 0.04475 -0.07335 rpy=6.12323e-17 -8.04912e-16 -3.52374e-15 -> xyz=-1.91513e-15 0.04475 -0.07335 rpy=3.33067e-16 -1.05818e-16 -2.03288e-16
- joint left_w1_0: origin xyz=-5.55112e-17 -0.0285 -0.13567 rpy=1.57652e-14 -1.23165e-16 1.11994e-14 -> xyz=-5.55112e-17 -0.0285 -0.13567 rpy=-4.71845e-16 3.45904e-15 -1.18829e-15
- joint left_w2_0: axis 1 0 0 -> -1 0 0; origin xyz=-0.0285 0.0285 -0.057 rpy=-3.36618e-14 -2.11528e-30 -6.12323e-17 -> xyz=0.0285 0.0285 -0.057 rpy=3.4972e-15 -8.32667e-17 -9.70669e-32
- joint right_e1_0: origin xyz=-0.04229 1.9082e-17 -0.289385 rpy=-1.09476e-47 7.39557e-32 1.2326e-32 -> xyz=-0.04229 1.47751e-17 -0.289385 rpy=1.07561e-45 7.39557e-32 1.84889e-32
- joint right_e2_0: origin xyz=0.03229 -6.93889e-18 -0.12429 rpy=3.03858e-64 4.93038e-32 1.2326e-32 -> xyz=0.04229 -1.56125e-17 -0.12429 rpy=3.03858e-64 4.93038e-32 1.2326e-32
- joint right_gripper_0: origin xyz=-0.0285 -6.93889e-18 -0.0335 rpy=3.03858e-64 4.93038e-32 1.2326e-32 -> xyz=0.0285 -6.93889e-18 -0.032251 rpy=-2.71671e-32 1.87354e-29 1.2326e-32
- joint right_s3_0: origin xyz=3.88578e-16 0.0323582 -0.07335 rpy=-2.73691e-48 4.93038e-32 4.71657e-48 -> xyz=3.88578e-16 0.04475 -0.07335 rpy=-1.08655e-45 -1.28919e-43 -6.16298e-33
- joint right_w2_0: origin xyz=0.0285 0.0285 -0.057 rpy=3.03858e-64 4.93038e-32 1.2326e-32 -> xyz=0.0285 0.0285 -0.057 rpy=7.5053e-62 -4.93038e-32 -3.14159

Commit message: fix right arm ik

File: almond_axol/kinematics/urdf/axol.urdf (robot description, URDF)
Before this commit: robot assembly, 19 links, 18 joints
Joints:
- joint right_e2_0: origin xyz=0.04229 -1.56125e-17 -0.12429 rpy=3.03858e-64 4.93038e-32 1.2326e-32 -> xyz=0.04229 -5.37817e-17 -0.12429 rpy=7.66335e-47 -2.46519e-32 3.14159
- joint right_gripper_0: origin xyz=0.0285 -6.93889e-18 -0.032251 rpy=-2.71671e-32 1.87354e-29 1.2326e-32 -> xyz=-0.0285 -7.09742e-18 -0.032251 rpy=2.46519e-32 1.4083e-43 -3.14159
- joint right_w1_0: axis 0 -1 0 -> 0 1 0; origin xyz=5.55112e-17 -0.0285 -0.13301 rpy=3.03858e-64 4.93038e-32 1.2326e-32 -> xyz=1.11022e-16 0.0285 -0.13567 rpy=1.09476e-47 2.55312e-94 -4.66423e-47
- joint right_w2_0: origin xyz=0.0285 0.0285 -0.057 rpy=7.5053e-62 -4.93038e-32 -3.14159 -> xyz=0.0285 -0.0285 -0.057 rpy=3.9443e-31 2.46519e-31 -1.30277e-45

Commit message: fix urdf

File: almond_axol/kinematics/urdf/axol.urdf (robot description, URDF)
Before this commit: robot assembly, 19 links, 18 joints
Links:
- link left_gripper: mass 0.00016575 -> 0.00042575; geometry collision mesh filename=package://assembly/meshes/Left_Gripper.stl scale=1 1 1; visual mesh filename=package://assembly/meshes/Left_Gripper.stl scale=1 1 1
- link right_gripper: mass 0.00016575 -> 0.00042575; geometry collision mesh filename=package://assembly/meshes/Right_Gripper.stl scale=1 1 1; visual mesh filename=package://assembly/meshes/Right_Gripper.stl scale=1 1 1
Joints:
- joint left_gripper_0: axis 0 0 -1 -> 0 0 1
- joint right_gripper_0: origin xyz=-0.0285 -7.09742e-18 -0.032251 rpy=2.46519e-32 1.4083e-43 -3.14159 -> xyz=0.0285 -7.09742e-18 -0.032251 rpy=0 -0 0
- joint right_w2_0: axis -1 0 0 -> 1 0 0; origin xyz=0.0285 -0.0285 -0.057 rpy=3.9443e-31 2.46519e-31 -1.30277e-45 -> xyz=0.0285 -0.0285 -0.057 rpy=-3.73315e-45 -4.43734e-31 3.14159

Commit message: read end stops

File: almond_axol/kinematics/urdf/axol.urdf (robot description, URDF)
Before this commit: robot assembly, 19 links, 18 joints
Joints:
- joint left_e1_0: limit lower=0.0 upper=2.6389 effort=87.0 velocity=30.0 -> lower=0.0 upper=2.6180 effort=87.0 velocity=30.0
- joint left_e2_0: limit lower=-1.5708 upper=1.5708 effort=87.0 velocity=30.0 -> lower=-2.3562 upper=2.3562 effort=87.0 velocity=30.0
- joint left_s1_0: limit lower=-1.5708 upper=1.5708 effort=87.0 velocity=30.0 -> lower=-1.5708 upper=3.1416 effort=87.0 velocity=30.0
- joint left_s2_0: limit lower=-1.5708 upper=0.1885 effort=87.0 velocity=30.0 -> lower=-0.3491 upper=3.1416 effort=87.0 velocity=30.0
- joint left_s3_0: limit lower=-1.5708 upper=1.5708 effort=87.0 velocity=30.0 -> lower=-2.3562 upper=2.3562 effort=87.0 velocity=30.0
- joint right_e1_0: limit lower=-2.6389 upper=0.0 effort=87.0 velocity=30.0 -> lower=-2.6180 upper=0.0 effort=87.0 velocity=30.0
- joint right_e2_0: limit lower=-1.5708 upper=1.5708 effort=87.0 velocity=30.0 -> lower=-2.3562 upper=2.3562 effort=87.0 velocity=30.0
- joint right_s1_0: limit lower=-1.5708 upper=1.5708 effort=87.0 velocity=30.0 -> lower=-1.5708 upper=3.1416 effort=87.0 velocity=30.0
- joint right_s2_0: limit lower=-0.1885 upper=1.5708 effort=87.0 velocity=30.0 -> lower=-3.1416 upper=0.3491 effort=87.0 velocity=30.0
- joint right_s3_0: limit lower=-1.5708 upper=1.5708 effort=87.0 velocity=30.0 -> lower=-2.3562 upper=2.3562 effort=87.0 velocity=30.0

Commit message: zero pos script

File: almond_axol/kinematics/urdf/axol.urdf (robot description, URDF)
Before this commit: robot assembly, 19 links, 18 joints
Joints:
- joint left_s2_0: limit lower=-0.3491 upper=3.1416 effort=87.0 velocity=30.0 -> lower=-3.1416 upper=0.3491 effort=87.0 velocity=30.0
- joint right_s1_0: limit lower=-1.5708 upper=3.1416 effort=87.0 velocity=30.0 -> lower=-3.1416 upper=1.5708 effort=87.0 velocity=30.0
- joint right_s2_0: limit lower=-3.1416 upper=0.3491 effort=87.0 velocity=30.0 -> lower=-0.3491 upper=3.1416 effort=87.0 velocity=30.0
