Commit message: Update URDF with actuated gripper and wire it into sim
Replace arm/gripper meshes and swap the fixed single-mesh gripper for the
new actuated gripper (prismatic finger joints, finger_b mimicking finger_a)
while preserving the existing arm link inertials, collision geometry, joint
limits, and naming. Add a dedicated *_gripper end-effector frame aligned with
*_w2 so teleop controller axes are unchanged, with the 90deg-rolled gripper
body hung off it via *_gripper_body. Map the normalized [0,1] gripper command
to the prismatic finger travel in sim teleop.

Co-authored-by: Cursor <cursoragent@cursor.com>

File: almond_axol/kinematics/urdf/axol.urdf (robot description, URDF)
Before this commit: robot assembly, 19 links, 18 joints
Links:
- added link left_gripper_body, mass 0.001; collision mesh filename=package://assembly/meshes/Gripper_Base.stl scale=1 1 1; visual mesh filename=package://assembly/meshes/Gripper_Base.stl scale=1 1 1
- added link left_gripper_finger_a, mass 0.001; collision mesh filename=package://assembly/meshes/Gripper_Tip.stl scale=1 1 1; visual mesh filename=package://assembly/meshes/Gripper_Tip.stl scale=1 1 1
- added link left_gripper_finger_b, mass 0.001; collision mesh filename=package://assembly/meshes/Gripper_Tip.stl scale=1 1 1; visual mesh filename=package://assembly/meshes/Gripper_Tip.stl scale=1 1 1
- added link right_gripper_body, mass 0.001; collision mesh filename=package://assembly/meshes/Gripper_Base.stl scale=1 1 1; visual mesh filename=package://assembly/meshes/Gripper_Base.stl scale=1 1 1
- added link right_gripper_finger_a, mass 0.001; collision mesh filename=package://assembly/meshes/Gripper_Tip.stl scale=1 1 1; visual mesh filename=package://assembly/meshes/Gripper_Tip.stl scale=1 1 1
- added link right_gripper_finger_b, mass 0.001; collision mesh filename=package://assembly/meshes/Gripper_Tip.stl scale=1 1 1; visual mesh filename=package://assembly/meshes/Gripper_Tip.stl scale=1 1 1
- link left_gripper: mass 0.00042575 -> 0.001; geometry 
- link right_gripper: mass 0.00042575 -> 0.001; geometry 
Joints:
- added joint left_gripper_body_0: type fixed, parent left_gripper, child left_gripper_body, origin xyz=0 0 0 rpy=1.5708 0 0, axis 0 0 1
- added joint left_gripper_joint_a: type prismatic, parent left_gripper_body, child left_gripper_finger_a, origin xyz=0.01256 -0.0508 -0.034 rpy=3.14159 -1.0297e-14 3.14159, axis 1 -8.38667e-15 1.67733e-14, limit lower=0.0 upper=0.058804 effort=20.0 velocity=1.0
- added joint left_gripper_joint_b: type prismatic, parent left_gripper_body, child left_gripper_finger_b, origin xyz=-0.01256 -0.0508 0.0325 rpy=0 1.12222e-14 -2.71556e-15, axis 1 -8.38667e-15 1.67733e-14, limit lower=0.0 upper=0.058804 effort=20.0 velocity=1.0, mimic joint=left_gripper_joint_a multiplier=1.0 offset=0.0
- added joint right_gripper_body_0: type fixed, parent right_gripper, child right_gripper_body, origin xyz=0 0 0 rpy=1.5708 0 0, axis 0 0 1
- added joint right_gripper_joint_a: type prismatic, parent right_gripper_body, child right_gripper_finger_a, origin xyz=0.01256 -0.0508 -0.034 rpy=3.14159 -1.0297e-14 3.14159, axis 1 -8.38667e-15 1.67733e-14, limit lower=0.0 upper=0.058804 effort=20.0 velocity=1.0
- added joint right_gripper_joint_b: type prismatic, parent right_gripper_body, child right_gripper_finger_b, origin xyz=-0.01256 -0.0508 0.0325 rpy=0 1.12222e-14 -2.71556e-15, axis 1 -8.38667e-15 1.67733e-14, limit lower=0.0 upper=0.058804 effort=20.0 velocity=1.0, mimic joint=right_gripper_joint_a multiplier=1.0 offset=0.0
- joint left_gripper_0: origin xyz=-0.0285 -7.09742e-18 -0.032251 rpy=9.71445e-17 -2.22045e-16 2.77556e-17 -> xyz=-0.0285 -2.55776e-17 -0.032251 rpy=0 0 0
- joint right_gripper_0: origin xyz=0.0285 -7.09742e-18 -0.032251 rpy=0 -0 0 -> xyz=0.0285 -1.5279e-17 -0.032251 rpy=0 0 0
