Commit message: Restore the longstanding Axol URDF
Remove the replacement CAD export and update IK, sim, teleop, and the WebXR overlay to use the historical 14-joint assembly model. Add frame/package contract tests and harden the Mantis tracking benchmark.

File: almond_axol/kinematics/urdf/axol.urdf (robot description, URDF)
Before this commit: robot axol_kit, 85 links, 84 joints
Links:
- removed link _zed_x_502__zed_x_50_lch_asm_din_en_iso7045_m2x5_4_8h_v1
- removed link _zed_x_502__zed_x_50_lch_asm_din_en_iso7045_m2x5_4_8h_v1_1
- removed link _zedx_mini_rev2__lower_case_v13
- removed link _zedx_mini_rev2__plastron_v2
- removed link _zedx_mini_rev2__plastron_v2_1
- removed link _zedx_mini_rev2__plastron_v2_2
- removed link _zedx_mini_rev2__upper_case_v8
- removed link bh_tx_mx_xx_xx
- removed link bh_tx_mx_xx_xx_1
- removed link bh_tx_mx_xx_xx_2
- removed link bh_tx_mx_xx_xx_3
- removed link camera_component___body_zed_x_one___front
- removed link camera_component___body_zed_x_one___front_1
- removed link camera_component___body_zed_x_one___rear
- removed link camera_component___body_zed_x_one___rear_1
- removed link camera_component___connector___fakra_plug
- removed link camera_component___connector___fakra_plug_1
- removed link camera_component___seal___zed_x_one
- removed link camera_component___seal___zed_x_one_1
- removed link fisheye_lens__1_
- removed link fisheye_lens__1__1
- removed link head_mount__1_
- removed link hexalobular_socket_head_cap_screw_iso14579_m2x0_4x10
- removed link hexalobular_socket_head_cap_screw_iso14579_m2x0_4x10_1
- removed link hexalobular_socket_head_cap_screw_iso14579_m2x0_4x10_2
- removed link hexalobular_socket_head_cap_screw_iso14579_m2x0_4x10_3
- removed link hexalobular_socket_head_cap_screw_iso14579_m2x0_4x10_4
- removed link hexalobular_socket_head_cap_screw_iso14579_m2x0_4x10_5
- removed link hexalobular_socket_head_cap_screw_iso14579_m2x0_4x10_6
- removed link hexalobular_socket_head_cap_screw_iso14579_m2x0_4x10_7
- removed link hexalobular_socket_pan_head_screw_iso_14583_m2x5
- removed link hexalobular_socket_pan_head_screw_iso_14583_m2x5_1
- removed link hexalobular_socket_pan_head_screw_iso_14583_m2x5_2
- removed link hexalobular_socket_pan_head_screw_iso_14583_m2x5_3
- removed link left_gripper_body
- removed link left_gripper_finger_a
- removed link left_gripper_finger_b
- removed link part_1
- removed link right_gripper_body
- removed link right_gripper_finger_a
- removed link right_gripper_finger_b
- removed link sh_hx_mx_xx_xx
- removed link sh_hx_mx_xx_xx_1
- removed link sh_hx_mx_xx_xx_10
- removed link sh_hx_mx_xx_xx_11
- removed link sh_hx_mx_xx_xx_12
- removed link sh_hx_mx_xx_xx_13
- removed link sh_hx_mx_xx_xx_14
- removed link sh_hx_mx_xx_xx_15
- removed link sh_hx_mx_xx_xx_2
- removed link sh_hx_mx_xx_xx_3
- removed link sh_hx_mx_xx_xx_4
- removed link sh_hx_mx_xx_xx_5
- removed link sh_hx_mx_xx_xx_6
- removed link sh_hx_mx_xx_xx_7
- removed link sh_hx_mx_xx_xx_8
- removed link sh_hx_mx_xx_xx_9
- removed link wrist_mount
- removed link wrist_mount_1
- removed link wrist_mount__1_
- removed link wrist_mount__2_
- removed link zed_xg120_asm_smb_jack_to_fakra_plug_adapter_v1
- removed link zed_xg120_asm_smb_jack_to_fakra_plug_adapter_v1_1
- removed link zed_xg120_asm_smb_jack_to_fakra_plug_adapter_v1_2
- removed link zed_xg120_asm_smb_jack_to_fakra_plug_adapter_v1_3
- removed link zed_xg120_asm_smb_jack_to_fakra_plug_adapter_v1_4
- link base: mass 0.02652 -> 0.02496; geometry collision mesh filename=package://assembly/meshes/Base.stl scale=1 1 1; visual mesh filename=package://assembly/meshes/Base.stl scale=1 1 1
- link left_e1: mass 5.60993 -> 0.00207775; geometry collision mesh filename=package://assembly/meshes/Left_E1.stl scale=1 1 1; visual mesh filename=package://assembly/meshes/Left_E1.stl scale=1 1 1
- link left_e2: mass 2.15214 -> 0.000797087; geometry collision mesh filename=package://assembly/meshes/Left_E2.stl scale=1 1 1; visual mesh filename=package://assembly/meshes/Left_E2.stl scale=1 1 1
- link left_gripper: mass 0.001 -> 0.00042575; geometry collision mesh filename=package://assembly/meshes/Left_Gripper.stl scale=1 1 1; visual mesh filename=package://assembly/meshes/Left_Gripper.stl scale=1 1 1
- link left_s2: mass 2.9365 -> 0.00108759; geometry collision mesh filename=package://assembly/meshes/Left_S2.stl scale=1 1 1; visual mesh filename=package://assembly/meshes/Left_S2.stl scale=1 1 1
- link left_s3: mass 2.08078 -> 0.000265068; geometry collision mesh filename=package://assembly/meshes/Left_S3.stl scale=1 1 1; visual mesh filename=package://assembly/meshes/Left_S3.stl scale=1 1 1
- link left_w0: mass 1.35486 -> 0.0005018; geometry collision mesh filename=package://assembly/meshes/Left_W0.stl scale=1 1 1; visual mesh filename=package://assembly/meshes/Left_W0.stl scale=1 1 1
- link left_w1: mass 0.892737 -> 0.000330643; geometry collision mesh filename=package://assembly/meshes/Left_W1.stl scale=1 1 1; visual mesh filename=package://assembly/meshes/Left_W1.stl scale=1 1 1
- link left_w2: mass 0.116987 -> 4.33287e-05; geometry collision mesh filename=package://assembly/meshes/Left_W2.stl scale=1 1 1; visual mesh filename=package://assembly/meshes/Left_W2.stl scale=1 1 1
- link right_e1: mass 5.60993 -> 0.00207775; geometry collision mesh filename=package://assembly/meshes/Right_E1.stl scale=1 1 1; visual mesh filename=package://assembly/meshes/Right_E1.stl scale=1 1 1
- link right_e2: mass 2.15214 -> 0.000797087; geometry collision mesh filename=package://assembly/meshes/Right_E2.stl scale=1 1 1; visual mesh filename=package://assembly/meshes/Right_E2.stl scale=1 1 1
- link right_gripper: mass 0.001 -> 0.00042575; geometry collision mesh filename=package://assembly/meshes/Right_Gripper.stl scale=1 1 1; visual mesh filename=package://assembly/meshes/Right_Gripper.stl scale=1 1 1
- link right_s2: mass 2.9365 -> 0.00108759; geometry collision mesh filename=package://assembly/meshes/Right_S2.stl scale=1 1 1; visual mesh filename=package://assembly/meshes/Right_S2.stl scale=1 1 1
- link right_s3: mass 2.08078 -> 0.000265068; geometry collision mesh filename=package://assembly/meshes/Right_S3.stl scale=1 1 1; visual mesh filename=package://assembly/meshes/Right_S3.stl scale=1 1 1
- link right_w0: mass 1.35486 -> 0.0005018; geometry collision mesh filename=package://assembly/meshes/Right_W0.stl scale=1 1 1; visual mesh filename=package://assembly/meshes/Right_W0.stl scale=1 1 1
- link right_w1: mass 0.892737 -> 0.000330643; geometry collision mesh filename=package://assembly/meshes/Right_W1.stl scale=1 1 1; visual mesh filename=package://assembly/meshes/Right_W1.stl scale=1 1 1
- link right_w2: mass 0.116987 -> 4.33287e-05; geometry collision mesh filename=package://assembly/meshes/Right_W2.stl scale=1 1 1; visual mesh filename=package://assembly/meshes/Right_W2.stl scale=1 1 1
- link s1: mass 0.00374359 -> 0.003744; geometry collision mesh filename=package://assembly/meshes/S1.stl scale=1 1 1; visual mesh filename=package://assembly/meshes/S1.stl scale=1 1 1
Joints:
- removed joint base
- removed joint fastened_1
- removed joint fastened_1_1
- removed joint fastened_1_2
- removed joint fastened_1_3
- removed joint fastened_2
- removed joint fastened_2_1
- removed joint fastened_2_2
- removed joint fastened_3
- removed joint fastened_3_1
- removed joint fastened_3_10
- removed joint fastened_3_11
- removed joint fastened_3_12
- removed joint fastened_3_2
- removed joint fastened_3_3
- removed joint fastened_3_4
- removed joint fastened_3_5
- removed joint fastened_3_6
- removed joint fastened_3_7
- removed joint fastened_3_8
- removed joint fastened_3_9
- removed joint fastened_4
- removed joint fastened_4_1
- removed joint fastened_4_2
- removed joint fastened_4_3
- removed joint fastened_4_4
- removed joint fastened_4_5
- removed joint fastened_4_6
- removed joint fastened_4_7
- removed joint fastened_5
- removed joint group_1_fastened_joint
- removed joint group_1_fastened_joint_1
- removed joint group_1_fastened_joint_10
- removed joint group_1_fastened_joint_11
- removed joint group_1_fastened_joint_12
- removed joint group_1_fastened_joint_13
- removed joint group_1_fastened_joint_14
- removed joint group_1_fastened_joint_15
- removed joint group_1_fastened_joint_16
- removed joint group_1_fastened_joint_17
- removed joint group_1_fastened_joint_18
- removed joint group_1_fastened_joint_19
- removed joint group_1_fastened_joint_2
- removed joint group_1_fastened_joint_20
- removed joint group_1_fastened_joint_21
- removed joint group_1_fastened_joint_22
- removed joint group_1_fastened_joint_23
- removed joint group_1_fastened_joint_24
- removed joint group_1_fastened_joint_25
- removed joint group_1_fastened_joint_26
- removed joint group_1_fastened_joint_27
- removed joint group_1_fastened_joint_28
- removed joint group_1_fastened_joint_29
- removed joint group_1_fastened_joint_3
- removed joint group_1_fastened_joint_30
- removed joint group_1_fastened_joint_4
- removed joint group_1_fastened_joint_5
- removed joint group_1_fastened_joint_6
- removed joint group_1_fastened_joint_7
- removed joint group_1_fastened_joint_8
- removed joint group_1_fastened_joint_9
- removed joint hanging_node_to_root_joint
- removed joint left_gripper_body_0
- removed joint left_gripper_joint_a
- removed joint left_gripper_joint_b
- removed joint right_gripper_body_0
- removed joint right_gripper_joint_a
- removed joint right_gripper_joint_b
- added joint base_0: type fixed, parent base, child s1, origin xyz=-2.79001e-17 6.93889e-18 -0.06 rpy=0 -1.06752e-16 0, axis 1.06752e-16 0 1
- added joint fixed_node_to_root_joint_0: type fixed, parent root, child base, origin xyz=-2.77556e-17 -6.93889e-18 0.86 rpy=0 0 1.5707963267948966, axis 0 0 1
- joint left_e1_0: limit lower=0.0 upper=2.618 effort=87.0 velocity=30.0 -> lower=0.0 upper=2.6180 effort=87.0 velocity=30.0; origin xyz=0.04229 3.83668e-17 -0.289385 rpy=6.27582e-14 1.30104e-17 5.77135e-18 -> xyz=0.04229 1.56381e-16 -0.289385 rpy=1.11022e-16 -4.93529e-16 -6.92805e-17
- joint left_e2_0: origin xyz=-0.04229 -7.12753e-18 -0.12429 rpy=-3.2474e-15 -6.33174e-17 -2.54576e-14 -> xyz=-0.04229 -1.48698e-17 -0.12429 rpy=-8.32667e-17 -6.33174e-17 7.22079e-17
- joint left_gripper_0: origin xyz=-0.0285 -2.55776e-17 -0.032251 rpy=0 0 0 -> xyz=-0.0285 -7.09742e-18 -0.032251 rpy=9.71445e-17 -2.22045e-16 2.77556e-17
- joint left_s1_0: origin xyz=0.108787 0.0137132 -0.06 rpy=6.43813e-31 -9.66752e-16 8.11935e-28 -> xyz=0.13 9.40122e-18 0.06 rpy=2.77556e-17 -1.02798e-15 1.32751e-21
- joint left_s2_0: origin xyz=0.06958 -0.04475 3.33067e-16 rpy=-8.54059e-31 1.28437e-14 -1.22465e-16 -> xyz=0.06958 -0.04475 4.44089e-16 rpy=2.498e-16 3.92274e-16 -2.48934e-16
- joint left_s3_0: origin xyz=-3.88578e-16 0.04475 -0.07335 rpy=5.06891e-29 6.12323e-17 -7.93161e-15 -> xyz=-1.91513e-15 0.04475 -0.07335 rpy=3.33067e-16 -1.05818e-16 -2.03288e-16
- joint left_w1_0: origin xyz=-8.32667e-17 -0.0285 -0.13567 rpy=-4.2466e-15 1.76757e-14 2.71935e-15 -> xyz=-5.55112e-17 -0.0285 -0.13567 rpy=-4.71845e-16 3.45904e-15 -1.18829e-15
- joint left_w2_0: origin xyz=0.0285 0.0285 -0.057 rpy=-2.21714e-14 1.79213e-44 1.61661e-30 -> xyz=0.0285 0.0285 -0.057 rpy=3.4972e-15 -8.32667e-17 -9.70669e-32
- joint right_e1_0: limit lower=-2.618 upper=0.0 effort=87.0 velocity=30.0 -> lower=-2.6180 upper=0.0 effort=87.0 velocity=30.0; origin xyz=-0.04229 1.60479e-17 -0.289385 rpy=-6.12323e-17 6.12323e-17 -6.12323e-17 -> xyz=-0.04229 1.47751e-17 -0.289385 rpy=1.07561e-45 7.39557e-32 1.84889e-32
- joint right_e2_0: origin xyz=0.04229 -3.11655e-17 -0.12429 rpy=1.61476e-27 -7.92016e-28 -3.14159 -> xyz=0.04229 -5.37817e-17 -0.12429 rpy=7.66335e-47 -2.46519e-32 3.14159
- joint right_gripper_0: origin xyz=0.0285 -1.5279e-17 -0.032251 rpy=0 0 0 -> xyz=0.0285 -7.09742e-18 -0.032251 rpy=0 -0 0
- joint right_s1_0: origin xyz=-0.151213 0.0137132 -0.06 rpy=-2.27247e-31 -2.31296e-16 7.35455e-16 -> xyz=-0.13 2.46215e-18 0.06 rpy=-4.76873e-49 -2.31296e-16 7.65788e-33
- joint right_s2_0: origin xyz=-0.06958 -0.04475 4.44089e-16 rpy=-5.61996e-30 -1.32163e-14 -3.9443e-31 -> xyz=-0.06958 -0.04475 4.44089e-16 rpy=-1.28654e-32 -9.17877e-18 -7.824e-17
- joint right_s3_0: origin xyz=4.16334e-16 0.04475 -0.07335 rpy=-2.235e-28 1.07364e-27 -3.41903e-14 -> xyz=3.88578e-16 0.04475 -0.07335 rpy=-1.08655e-45 -1.28919e-43 -6.16298e-33
- joint right_w1_0: origin xyz=1.66533e-16 0.0285 -0.13567 rpy=9.03554e-29 -4.3255e-14 -4.98658e-30 -> xyz=1.11022e-16 0.0285 -0.13567 rpy=1.09476e-47 2.55312e-94 -4.66423e-47
- joint right_w2_0: origin xyz=0.0285 -0.0285 -0.057 rpy=-8.07794e-27 1.05707e-27 -3.14159 -> xyz=0.0285 -0.0285 -0.057 rpy=-3.73315e-45 -4.43734e-31 3.14159
