Commit message: Axol Mobile: fix right-arm rest pose, put the ground under the wheels
The right arm swung up out of its rest pose in sim. Three causes:

- pyroki's segment-to-segment routine pairs mismatched points for
  (anti)parallel segments, so the right upper arm hanging beside the lift
  column read 249 mm of clearance instead of 84 mm. Patch in a
  parallel-safe (Ericson) routine at import; a test flags when the
  almond-pyroki fork has the fix and the patch can go.
- The upper-arm guard allowed "at most 20 mm closer than home", which
  was calibrated on the classic stand where the capsules overlap at home.
  The default rest pose is 26 mm closer to the Jelly column than home, so
  cap the floor at zero: where the body is clear at home the guard stops
  actual contact. Classic floors are unchanged.
- The closed fingers' minimum-cylinder fit was ambiguous and landed on
  different axes per hand. Use an explicit collision cylinder along the
  jaw axis, sized over the full finger stroke (covers open fingers too).

Rebuilt from the wheeled Onshape export (separate wheel meshes; lift
stages now exactly 0-0.34 m). Adds a floor frame under the wheels; the
sim and the rest-pose viewer draw their ground plane there while the
IK world frame stays the classic one.

Co-Authored-By: Claude Opus 5.5 <noreply@anthropic.com>

File: almond_axol/kinematics/urdf/axol_mobile.urdf (robot description, URDF)
Before this commit: robot assembly, 26 links, 25 joints
Links:
- added link floor
- link left_fingers: geometry collision cylinder length=0.15216 radius=0.05876; visual mesh filename=package://assembly/meshes/mobile/left_fingers_0.stl scale=1 1 1
- link right_fingers: geometry collision cylinder length=0.15206 radius=0.05876; visual mesh filename=package://assembly/meshes/mobile/right_fingers_0.stl scale=1 1 1
Joints:
- added joint floor_0: type fixed, parent root, child floor, origin xyz=-0.112228 5.12225e-06 -0.46944 rpy=0 0 0
