Commit message: Whole-body IK switch: Jelly base and lift as IK joints
Arm IK stays the default: only the 14 arm joints move and the mobile
model is unchanged. kinematics.whole_body (panel: Kinematics ->
"Whole-body IK (sim only)") switches to a second generated model,
axol_mobile_whole_body.urdf, that roots the same torso and arms on the
Jelly's planar base (base_x, base_y, base_yaw about the Jelly centre)
and its lift (lift, 0 = fully raised; the second stage mimics it). Its
world frame is the arm model's at body zero, so poses agree at startup.

- Generator: builds both models from one set of visual meshes; collision
  is assembled per model from named pieces. Whole-body splits the column
  by stage (base / lift_stage / jelly) and covers the deck with three
  capsule strips; the arm model is numerically unchanged.
- Solver: body joints follow the arms in the public vector
  (BODY_JOINTS). They are held still while both hands are within
  comfortable reach (body_reach_start) and released smoothly beyond it,
  have their own step budgets and damping, no posture attractor, and no
  reach clamp. Shoulders are recomputed from each seed. Manipulability
  is measured over each arm's own joints.
- Fix: the collision-safe step zeroed the whole step when any joint sat
  on a limit and was pushed further out (whole-body starts with the lift
  on its raised limit). Only that component is dropped now.
- Teleop: reset keeps the base and lift where they are; the core exposes
  the body target and the sim renders it. Whole-body refuses to start on
  real hardware, in absolute (Mantis) mode and in data collection.

Arm-mode IK matches the previous commit within float rounding (median
1e-7 rad over 300 random single solves).

Co-Authored-By: Claude Opus 5.5 <noreply@anthropic.com>

File: almond_axol/kinematics/urdf/axol_mobile_whole_body.urdf (robot description, URDF)
Before this commit: robot assembly, 28 links, 27 joints
Links:
- added link base_x_link
- added link base_y_link
- added link deck_0; collision cylinder length=0.606 radius=0.14516
- added link deck_1; collision cylinder length=0.606 radius=0.14516
- added link deck_2; collision cylinder length=0.606 radius=0.14516
- added link world
- link base: geometry collision mesh filename=package://assembly/meshes/mobile/base_whole_body_collision.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 scale=1 1 1; visual mesh filename=package://assembly/meshes/mobile/base_0.stl scale=1 1 1
- link jelly: geometry collision mesh filename=package://assembly/meshes/mobile/jelly_whole_body_collision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 scale=1 1 1; visual mesh filename=package://assembly/meshes/mobile/jelly_0.stl scale=1 1 1
- link lift_stage: geometry collision mesh filename=package://assembly/meshes/mobile/lift_stage_whole_body_coll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 scale=1 1 1; visual mesh filename=package://assembly/meshes/mobile/lift_stage_0.stl scale=1 1 1
Joints:
- removed joint jelly_0
- removed joint lift_stage_0
- added joint base_x: type prismatic, parent world, child base_x_link, origin xyz=-0.112228 5.12225e-06 -0.46944 rpy=0 0 0, axis 1 0 0, limit lower=-10 upper=10 effort=1 velocity=1
- added joint base_y: type prismatic, parent base_x_link, child base_y_link, origin xyz=0 0 0 rpy=0 0 0, axis 0 1 0, limit lower=-10 upper=10 effort=1 velocity=1
- added joint base_yaw: type revolute, parent base_y_link, child jelly, origin xyz=0 0 0 rpy=0 0 0, axis 0 0 1, limit lower=-6.28319 upper=6.28319 effort=1 velocity=1
- added joint deck_0_0: type fixed, parent jelly, child deck_0, origin xyz=0 0 0 rpy=0 0 0
- added joint deck_1_0: type fixed, parent jelly, child deck_1, origin xyz=0 0 0 rpy=0 0 0
- added joint deck_2_0: type fixed, parent jelly, child deck_2, origin xyz=0 0 0 rpy=0 0 0
- added joint lift: type prismatic, parent jelly, child lift_stage, origin xyz=0 0 0 rpy=0 0 0, axis 0 0 -1, limit lower=0 upper=0.34 effort=1 velocity=1
- added joint lift_2: type prismatic, parent lift_stage, child root, origin xyz=0.112228 -5.12225e-06 0.46944 rpy=0 0 0, axis 0 0 -1, limit lower=0 upper=0.34 effort=1 velocity=1, mimic joint=lift multiplier=1 offset=0
- joint floor_0: parent root -> world
