Commit message: Sim URDF: drive gains as <drive> on each arm joint
Drop axol_jelly_sim_drives.json; the motors' kp/kd now travel with the
model as a custom <drive stiffness damping> element next to <dynamics>.

Co-Authored-By: Claude Opus 5.5 <noreply@anthropic.com>

File: almond_axol/kinematics/urdf/axol_jelly_sim.urdf (robot description, URDF)
Before this commit: robot assembly, 37 links, 36 joints
Joints:
- joint head_camera_left_optical_0: origin xyz=0.0250101 -0.107619 0.132221 rpy=-2.61799 -2.03277e-06 -3.14159 -> xyz=0.0250101 -0.104017 0.138461 rpy=-2.61799 -2.03277e-06 -3.14159
- joint head_camera_right_optical_0: origin xyz=-0.0249785 -0.107619 0.132221 rpy=-2.61799 -2.03277e-06 -3.14159 -> xyz=-0.0249785 -0.104017 0.138461 rpy=-2.61799 -2.03277e-06 -3.14159
