Commit message: Wrist camera frames: fix the roll, flag the origin
Rendering the wrist view from axol_jelly_sim.urdf put the gripper at the
top of the image; real wrist frames show it at the bottom with the
fingers pointing up into the scene. The roll, which the square camera
body leaves undetermined in the CAD, had been guessed from the gripper's
jaw axis and was 180 degrees off. It is now set so +y (image down) points
from the lens toward that gripper's fingers; a test pins it.

The frames' origin stays at the camera body's seal ring, which is not the
optical centre (the ZED X One S fisheye's projection centre is somewhere
forward inside the lens and is not published). Every Jelly URDF's header
now says so, pending a calibrated offset.

Co-Authored-By: Claude Opus 5.5 <noreply@anthropic.com>

File: almond_axol/kinematics/urdf/axol_jelly.urdf (robot description, URDF)
Before this commit: robot assembly, 40 links, 39 joints
Joints:
- joint left_wrist_camera_optical_0: origin xyz=2.24535e-06 -0.0919574 -0.0450941 rpy=-2.70526 -2.78718e-06 -1.29967e-06 -> xyz=2.24535e-06 -0.0919574 -0.0450941 rpy=2.70526 7.56894e-06 -3.14158
- joint right_wrist_camera_optical_0: origin xyz=2.11683e-06 -0.091963 -0.0450936 rpy=-2.70526 5.02791e-06 2.34453e-06 -> xyz=2.11683e-06 -0.091963 -0.0450936 rpy=2.70526 -6.68559e-06 3.14159

File: almond_axol/kinematics/urdf/axol_jelly_sim.urdf (robot description, URDF)
Before this commit: robot assembly, 37 links, 36 joints
Joints:
- joint left_wrist_camera_optical_0: origin xyz=2.24535e-06 -0.0919574 -0.0450941 rpy=-2.70526 -2.78718e-06 -1.29967e-06 -> xyz=2.24535e-06 -0.0919574 -0.0450941 rpy=2.70526 7.56894e-06 -3.14158
- joint right_wrist_camera_optical_0: origin xyz=2.11683e-06 -0.091963 -0.0450936 rpy=-2.70526 5.02791e-06 2.34453e-06 -> xyz=2.11683e-06 -0.091963 -0.0450936 rpy=2.70526 -6.68559e-06 3.14159

File: almond_axol/kinematics/urdf/axol_jelly_whole_body.urdf (robot description, URDF)
Before this commit: robot assembly, 46 links, 45 joints
Joints:
- joint left_wrist_camera_optical_0: origin xyz=2.24535e-06 -0.0919574 -0.0450941 rpy=-2.70526 -2.78718e-06 -1.29967e-06 -> xyz=2.24535e-06 -0.0919574 -0.0450941 rpy=2.70526 7.56894e-06 -3.14158
- joint right_wrist_camera_optical_0: origin xyz=2.11683e-06 -0.091963 -0.0450936 rpy=-2.70526 5.02791e-06 2.34453e-06 -> xyz=2.11683e-06 -0.091963 -0.0450936 rpy=2.70526 -6.68559e-06 3.14159

Commit message: Wrist camera frames: optical centre from Stereolabs' lens frame
The wrist optical frames sat at the camera body's seal ring, ~19 mm
behind the ZED X One S fisheye's projection centre, which shrank and
shifted the gripper in wrist renders by tens of pixels.

The origin is now Stereolabs' fisheye-lens reference frame from the
camera's own CAD (on the lens axis, 18.9 mm ahead of the ring). It was
checked against real frames from both wrist cameras on a Jelly robot
(no arm motion): projecting the gripper through each camera's factory
calibration (ZED SDK Kannala-Brandt intrinsics) and fitting the depth
put the projection centre +19.0-19.5 mm ahead of the ring, and +0.0 /
+0.5 mm from the new origin after the change. The generator checks the
lens frame sits on the axis at a plausible depth.

Co-Authored-By: Claude Opus 5.5 <noreply@anthropic.com>

File: almond_axol/kinematics/urdf/axol_jelly.urdf (robot description, URDF)
Before this commit: robot assembly, 40 links, 39 joints
Joints:
- joint left_wrist_camera_optical_0: origin xyz=2.24535e-06 -0.0919574 -0.0450941 rpy=2.70526 7.56894e-06 -3.14158 -> xyz=2.3035e-06 -0.0839662 -0.0622315 rpy=2.70526 7.56894e-06 -3.14158
- joint right_wrist_camera_optical_0: origin xyz=2.11683e-06 -0.091963 -0.0450936 rpy=2.70526 -6.68559e-06 3.14159 -> xyz=2.01193e-06 -0.0839718 -0.0622309 rpy=2.70526 -6.68559e-06 3.14159

File: almond_axol/kinematics/urdf/axol_jelly_sim.urdf (robot description, URDF)
Before this commit: robot assembly, 37 links, 36 joints
Joints:
- joint left_wrist_camera_optical_0: origin xyz=2.24535e-06 -0.0919574 -0.0450941 rpy=2.70526 7.56894e-06 -3.14158 -> xyz=2.3035e-06 -0.0839662 -0.0622315 rpy=2.70526 7.56894e-06 -3.14158
- joint right_wrist_camera_optical_0: origin xyz=2.11683e-06 -0.091963 -0.0450936 rpy=2.70526 -6.68559e-06 3.14159 -> xyz=2.01193e-06 -0.0839718 -0.0622309 rpy=2.70526 -6.68559e-06 3.14159

File: almond_axol/kinematics/urdf/axol_jelly_whole_body.urdf (robot description, URDF)
Before this commit: robot assembly, 46 links, 45 joints
Joints:
- joint left_wrist_camera_optical_0: origin xyz=2.24535e-06 -0.0919574 -0.0450941 rpy=2.70526 7.56894e-06 -3.14158 -> xyz=2.3035e-06 -0.0839662 -0.0622315 rpy=2.70526 7.56894e-06 -3.14158
- joint right_wrist_camera_optical_0: origin xyz=2.11683e-06 -0.091963 -0.0450936 rpy=2.70526 -6.68559e-06 3.14159 -> xyz=2.01193e-06 -0.0839718 -0.0622309 rpy=2.70526 -6.68559e-06 3.14159

Commit message: Wrist camera frames: projection centre from Stereolabs' camera model
Stereolabs' STEP model of the ZED X One S fisheye includes the camera's
optics, which the robot's Onshape export drops: an "Image plane", an
infrared filter and a "Simple FOV" solid whose bounding planes meet on
the lens axis at z = 10.696 mm in the camera's CAD frame (2.2 mm behind
the front glass, 23.3 mm ahead of the body's seal ring). That is where
the camera's rays converge, so the wrist optical origin is now there
(PROJECTION_CENTRE_Z, placed from the export's zed_x_one_gs_compact
frame, which is the same CAD origin and axes).

It replaces the lens part's own modelling origin (4.4 mm further back).
Fitting real wrist images through each camera's factory calibration
cannot tell the two apart (the overlap is flat to within ~3 mm: left
-1..+2 mm, right +1..+4 mm around the old frame), so the explicit model
wins.

Co-Authored-By: Claude Opus 5.5 <noreply@anthropic.com>

File: almond_axol/kinematics/urdf/axol_jelly.urdf (robot description, URDF)
Before this commit: robot assembly, 40 links, 39 joints
Joints:
- joint left_wrist_camera_optical_0: origin xyz=2.3035e-06 -0.0839662 -0.0622315 rpy=2.70526 7.56894e-06 -3.14158 -> xyz=2.33373e-06 -0.0821122 -0.0662075 rpy=2.70526 7.56894e-06 -3.14158
- joint right_wrist_camera_optical_0: origin xyz=2.01193e-06 -0.0839718 -0.0622309 rpy=2.70526 -6.68559e-06 3.14159 -> xyz=2.00434e-06 -0.0821178 -0.066207 rpy=2.70526 -6.68559e-06 3.14159

File: almond_axol/kinematics/urdf/axol_jelly_sim.urdf (robot description, URDF)
Before this commit: robot assembly, 37 links, 36 joints
Joints:
- joint left_wrist_camera_optical_0: origin xyz=2.3035e-06 -0.0839662 -0.0622315 rpy=2.70526 7.56894e-06 -3.14158 -> xyz=2.33373e-06 -0.0821122 -0.0662075 rpy=2.70526 7.56894e-06 -3.14158
- joint right_wrist_camera_optical_0: origin xyz=2.01193e-06 -0.0839718 -0.0622309 rpy=2.70526 -6.68559e-06 3.14159 -> xyz=2.00434e-06 -0.0821178 -0.066207 rpy=2.70526 -6.68559e-06 3.14159

File: almond_axol/kinematics/urdf/axol_jelly_whole_body.urdf (robot description, URDF)
Before this commit: robot assembly, 46 links, 45 joints
Joints:
- joint left_wrist_camera_optical_0: origin xyz=2.3035e-06 -0.0839662 -0.0622315 rpy=2.70526 7.56894e-06 -3.14158 -> xyz=2.33373e-06 -0.0821122 -0.0662075 rpy=2.70526 7.56894e-06 -3.14158
- joint right_wrist_camera_optical_0: origin xyz=2.01193e-06 -0.0839718 -0.0622309 rpy=2.70526 -6.68559e-06 3.14159 -> xyz=2.00434e-06 -0.0821178 -0.066207 rpy=2.70526 -6.68559e-06 3.14159

Commit message: Head camera frames: projection centre from Stereolabs' camera model
Each ZED X Mini Wide lens's FOV solid meets on its axis 7.2 mm behind the
lens cover's mid-plane (ZED_X_Mini_Wide.step); move both head optical
frames there from the cover centre.

Co-Authored-By: Claude Opus 5.5 <noreply@anthropic.com>

File: almond_axol/kinematics/urdf/axol_jelly.urdf (robot description, URDF)
Before this commit: robot assembly, 40 links, 39 joints
Joints:
- joint head_camera_left_optical_0: origin xyz=0.0250101 -0.107619 0.132221 rpy=-2.61799 -2.03277e-06 -3.14159 -> xyz=0.0250101 -0.104017 0.138461 rpy=-2.61799 -2.03277e-06 -3.14159
- joint head_camera_right_optical_0: origin xyz=-0.0249785 -0.107619 0.132221 rpy=-2.61799 -2.03277e-06 -3.14159 -> xyz=-0.0249785 -0.104017 0.138461 rpy=-2.61799 -2.03277e-06 -3.14159

File: almond_axol/kinematics/urdf/axol_jelly_whole_body.urdf (robot description, URDF)
Before this commit: robot assembly, 46 links, 45 joints
Joints:
- joint head_camera_left_optical_0: origin xyz=0.0250101 -0.107619 0.132221 rpy=-2.61799 -2.03277e-06 -3.14159 -> xyz=0.0250101 -0.104017 0.138461 rpy=-2.61799 -2.03277e-06 -3.14159
- joint head_camera_right_optical_0: origin xyz=-0.0249785 -0.107619 0.132221 rpy=-2.61799 -2.03277e-06 -3.14159 -> xyz=-0.0249785 -0.104017 0.138461 rpy=-2.61799 -2.03277e-06 -3.14159

Commit message: Jelly URDFs: regenerate from the export with the fixed gripper tips
Gripper_Tip reshaped (69.0 -> 54.8 cm3) and placed 11 mm further out on
each finger; finger joints' closed origin moves 0.19 mm. Finger visuals
keep the full CAD mesh (no simplification within 0.3 mm); the IK finger
cylinders shorten 152 -> 130 mm. Other meshes are unchanged.

Co-Authored-By: Claude Opus 5.5 <noreply@anthropic.com>

File: almond_axol/kinematics/urdf/axol_jelly.urdf (robot description, URDF)
Before this commit: robot assembly, 40 links, 39 joints
Links:
- link left_fingers: geometry collision cylinder length=0.1299 radius=0.05876
- link right_fingers: geometry collision cylinder length=0.13015 radius=0.05876
Joints:
- joint floor_0: origin xyz=-0.112228 5.12225e-06 -0.46944 rpy=0 0 0 -> xyz=-0.112228 5.24549e-06 -0.46944 rpy=0 0 0
- joint head_camera_left_optical_0: origin xyz=0.0250101 -0.104017 0.138461 rpy=-2.61799 -2.03277e-06 -3.14159 -> xyz=0.0250102 -0.104017 0.138461 rpy=-2.61799 -2.03277e-06 -3.14159
- joint head_camera_right_optical_0: origin xyz=-0.0249785 -0.104017 0.138461 rpy=-2.61799 -2.03277e-06 -3.14159 -> xyz=-0.0249784 -0.104017 0.138461 rpy=-2.61799 -2.03277e-06 -3.14159
- joint jelly_0: origin xyz=-0.112228 5.12225e-06 -0.46944 rpy=0 0 0 -> xyz=-0.112228 5.24549e-06 -0.46944 rpy=0 0 0
- joint left_finger_1_0: origin xyz=0.0123745 0.0340885 -0.0542893 rpy=1.5708 -2.65359e-06 -3.14159 -> xyz=0.0125619 0.0340885 -0.0542893 rpy=1.57079 -2.65359e-06 -3.14159
- joint left_finger_2_0: origin xyz=-0.0123708 -0.0324116 -0.0542893 rpy=1.5708 -3.74129e-12 4.69282e-06 -> xyz=-0.0125578 -0.0324116 -0.0542893 rpy=1.5708 -3.76379e-12 4.69282e-06
- joint left_wrist_camera_optical_0: origin xyz=2.33373e-06 -0.0821122 -0.0662075 rpy=2.70526 7.56894e-06 -3.14158 -> xyz=2.45697e-06 -0.0821122 -0.0662075 rpy=2.70526 7.56617e-06 -3.14158
- joint lift_stage_0: origin xyz=-0.112228 5.12225e-06 -0.46944 rpy=0 0 0 -> xyz=-0.112228 5.24549e-06 -0.46944 rpy=0 0 0
- joint right_finger_1_0: origin xyz=0.0125623 0.0340828 -0.0542888 rpy=1.57079 -9.99998e-06 3.14159 -> xyz=0.0125624 0.0340829 -0.0542888 rpy=1.5708 -1e-05 -3.14159
- joint right_finger_2_0: origin xyz=-0.0125578 -0.0324171 -0.0542887 rpy=1.5708 7.34639e-06 -2.03923e-06 -> xyz=-0.0125574 -0.0324172 -0.0542887 rpy=1.5708 7.34641e-06 3.26795e-06
- joint right_wrist_camera_optical_0: origin xyz=2.00434e-06 -0.0821178 -0.066207 rpy=2.70526 -6.68559e-06 3.14159 -> xyz=2.70961e-06 -0.0821178 -0.066207 rpy=2.70526 -6.68623e-06 -3.14159
- joint wheel_1_link_0: origin xyz=0.215832 0.215834 0.06335 rpy=3.14159 0 5.30718e-06 -> xyz=0.215834 0.215832 0.06335 rpy=3.14159 0 0
- joint wheel_2_link_0: origin xyz=0.215834 -0.215832 0.06335 rpy=0 0 0 -> xyz=0.215832 -0.215834 0.06335 rpy=0 0 -5.30718e-06
- joint wheel_3_link_0: origin xyz=-0.215834 0.215832 0.06335 rpy=0 0 0 -> xyz=-0.215832 0.215834 0.06335 rpy=0 0 0
- joint wheel_4_link_0: origin xyz=-0.215832 -0.215834 0.06335 rpy=3.14159 0 5.30718e-06 -> xyz=-0.215834 -0.215832 0.06335 rpy=3.14159 0 0

File: almond_axol/kinematics/urdf/axol_jelly_sim.urdf (robot description, URDF)
Before this commit: robot assembly, 37 links, 36 joints
Joints:
- joint head_camera_left_optical_0: origin xyz=0.0250101 -0.104017 0.138461 rpy=-2.61799 -2.03277e-06 -3.14159 -> xyz=0.0250102 -0.104017 0.138461 rpy=-2.61799 -2.03277e-06 -3.14159
- joint head_camera_right_optical_0: origin xyz=-0.0249785 -0.104017 0.138461 rpy=-2.61799 -2.03277e-06 -3.14159 -> xyz=-0.0249784 -0.104017 0.138461 rpy=-2.61799 -2.03277e-06 -3.14159
- joint left_finger_1_joint: origin xyz=0.0123745 0.0340885 -0.0542893 rpy=1.5708 -2.65359e-06 -3.14159 -> xyz=0.0125619 0.0340885 -0.0542893 rpy=1.57079 -2.65359e-06 -3.14159
- joint left_finger_2_joint: origin xyz=-0.0123708 -0.0324116 -0.0542893 rpy=1.5708 -3.74129e-12 4.69282e-06 -> xyz=-0.0125578 -0.0324116 -0.0542893 rpy=1.5708 -3.76379e-12 4.69282e-06
- joint left_wrist_camera_optical_0: origin xyz=2.33373e-06 -0.0821122 -0.0662075 rpy=2.70526 7.56894e-06 -3.14158 -> xyz=2.45697e-06 -0.0821122 -0.0662075 rpy=2.70526 7.56617e-06 -3.14158
- joint lift_2: origin xyz=0.112228 -5.12225e-06 0.46944 rpy=0 0 0 -> xyz=0.112228 -5.24549e-06 0.46944 rpy=0 0 0
- joint right_finger_1_joint: origin xyz=0.0125623 0.0340828 -0.0542888 rpy=1.57079 -9.99998e-06 3.14159 -> xyz=0.0125624 0.0340829 -0.0542888 rpy=1.5708 -1e-05 -3.14159
- joint right_finger_2_joint: origin xyz=-0.0125578 -0.0324171 -0.0542887 rpy=1.5708 7.34639e-06 -2.03923e-06 -> xyz=-0.0125574 -0.0324172 -0.0542887 rpy=1.5708 7.34641e-06 3.26795e-06
- joint right_wrist_camera_optical_0: origin xyz=2.00434e-06 -0.0821178 -0.066207 rpy=2.70526 -6.68559e-06 3.14159 -> xyz=2.70961e-06 -0.0821178 -0.066207 rpy=2.70526 -6.68623e-06 -3.14159
- joint wheel_1: origin xyz=0.215832 0.215834 0.06335 rpy=3.14159 0 5.30718e-06 -> xyz=0.215834 0.215832 0.06335 rpy=3.14159 0 0
- joint wheel_2: origin xyz=0.215834 -0.215832 0.06335 rpy=0 0 0 -> xyz=0.215832 -0.215834 0.06335 rpy=0 0 -5.30718e-06
- joint wheel_3: origin xyz=-0.215834 0.215832 0.06335 rpy=0 0 0 -> xyz=-0.215832 0.215834 0.06335 rpy=0 0 0
- joint wheel_4: origin xyz=-0.215832 -0.215834 0.06335 rpy=3.14159 0 5.30718e-06 -> xyz=-0.215834 -0.215832 0.06335 rpy=3.14159 0 0

File: almond_axol/kinematics/urdf/axol_jelly_whole_body.urdf (robot description, URDF)
Before this commit: robot assembly, 46 links, 45 joints
Links:
- link left_fingers: geometry collision cylinder length=0.1299 radius=0.05876
- link right_fingers: geometry collision cylinder length=0.13015 radius=0.05876
Joints:
- joint base_x: origin xyz=-0.112228 5.12225e-06 -0.46944 rpy=0 0 0 -> xyz=-0.112228 5.24549e-06 -0.46944 rpy=0 0 0
- joint floor_0: origin xyz=-0.112228 5.12225e-06 -0.46944 rpy=0 0 0 -> xyz=-0.112228 5.24549e-06 -0.46944 rpy=0 0 0
- joint head_camera_left_optical_0: origin xyz=0.0250101 -0.104017 0.138461 rpy=-2.61799 -2.03277e-06 -3.14159 -> xyz=0.0250102 -0.104017 0.138461 rpy=-2.61799 -2.03277e-06 -3.14159
- joint head_camera_right_optical_0: origin xyz=-0.0249785 -0.104017 0.138461 rpy=-2.61799 -2.03277e-06 -3.14159 -> xyz=-0.0249784 -0.104017 0.138461 rpy=-2.61799 -2.03277e-06 -3.14159
- joint left_finger_1_0: origin xyz=0.0123745 0.0340885 -0.0542893 rpy=1.5708 -2.65359e-06 -3.14159 -> xyz=0.0125619 0.0340885 -0.0542893 rpy=1.57079 -2.65359e-06 -3.14159
- joint left_finger_2_0: origin xyz=-0.0123708 -0.0324116 -0.0542893 rpy=1.5708 -3.74129e-12 4.69282e-06 -> xyz=-0.0125578 -0.0324116 -0.0542893 rpy=1.5708 -3.76379e-12 4.69282e-06
- joint left_wrist_camera_optical_0: origin xyz=2.33373e-06 -0.0821122 -0.0662075 rpy=2.70526 7.56894e-06 -3.14158 -> xyz=2.45697e-06 -0.0821122 -0.0662075 rpy=2.70526 7.56617e-06 -3.14158
- joint lift_2: origin xyz=0.112228 -5.12225e-06 0.46944 rpy=0 0 0 -> xyz=0.112228 -5.24549e-06 0.46944 rpy=0 0 0
- joint right_finger_1_0: origin xyz=0.0125623 0.0340828 -0.0542888 rpy=1.57079 -9.99998e-06 3.14159 -> xyz=0.0125624 0.0340829 -0.0542888 rpy=1.5708 -1e-05 -3.14159
- joint right_finger_2_0: origin xyz=-0.0125578 -0.0324171 -0.0542887 rpy=1.5708 7.34639e-06 -2.03923e-06 -> xyz=-0.0125574 -0.0324172 -0.0542887 rpy=1.5708 7.34641e-06 3.26795e-06
- joint right_wrist_camera_optical_0: origin xyz=2.00434e-06 -0.0821178 -0.066207 rpy=2.70526 -6.68559e-06 3.14159 -> xyz=2.70961e-06 -0.0821178 -0.066207 rpy=2.70526 -6.68623e-06 -3.14159
- joint wheel_1_link_0: origin xyz=0.215832 0.215834 0.06335 rpy=3.14159 0 5.30718e-06 -> xyz=0.215834 0.215832 0.06335 rpy=3.14159 0 0
- joint wheel_2_link_0: origin xyz=0.215834 -0.215832 0.06335 rpy=0 0 0 -> xyz=0.215832 -0.215834 0.06335 rpy=0 0 -5.30718e-06
- joint wheel_3_link_0: origin xyz=-0.215834 0.215832 0.06335 rpy=0 0 0 -> xyz=-0.215832 0.215834 0.06335 rpy=0 0 0
- joint wheel_4_link_0: origin xyz=-0.215832 -0.215834 0.06335 rpy=3.14159 0 5.30718e-06 -> xyz=-0.215834 -0.215832 0.06335 rpy=3.14159 0 0
