Commit message: One URDF per Axol version: IK, viewers and simulators share one full model
The generated versions are now one file each — axol_standalone,
axol_ox_cart, axol_owl, axol_jelly, and axol_jelly_parcel for the parcel
gripper — next to the legacy axol.urdf. The Jelly arm-IK, whole-body and
sim files are merged into axol_jelly.urdf (and likewise for parcel).

Each file is the full robot: every moving part a joint (the Jelly base in
the plane and its two-stage lift, the Ox cart's lift, fingers or parcel
plate, wheels), AxolConfig's arm masses with estimates elsewhere, friction
and drive gains, per-part contact hulls in <collision>, and relative mesh
paths. With every body joint at zero the torso is the world origin, so IK
frames and recorded poses are unchanged. IK loads it through
kinematics.model.ik_urdf, which freezes the joints it does not solve (arm
IK: all but the arms; whole-body IK: plus base and lift) and collides the
capsule-friendly <ik_collision> pieces instead.

Jelly arm IK now collides the lift column per section (the whole-body
split) rather than one hull over all three: 96 pairs instead of 64, ~0.7 ms
more per solve. The full models' own masses weigh the arms exactly as
gravity compensation's tuned model (checked in MuJoCo with fusestatic off).

The generator is renamed scripts/build_urdfs.py and models each body's IK
and physics collision sets, lift and masses on its Body.

Co-Authored-By: Claude Opus 5.5 <noreply@anthropic.com>

File: almond_axol/kinematics/urdf/axol_jelly.urdf (robot description, URDF)
Before this commit: robot assembly, 40 links, 39 joints
Links:
- added link base_x_link, mass 0.01
- added link base_y_link, mass 0.01
- added link deck_0
- added link deck_1
- added link deck_2
- added link world
- link base: mass 0.02496 -> 4; geometry collision mesh filename=meshes/jelly/base__column_top_collision.stl scale=1 1 1; visual mesh filename=meshes/jelly/base_0.stl scale=1 1 1
- link head: mass None -> 0.3; geometry collision mesh filename=meshes/jelly/head_collision.stl scale=1 1 1; visual mesh filename=meshes/jelly/head_0.stl scale=1 1 1
- link jelly: mass None -> 40; geometry collision mesh filename=meshes/jelly/jelly__column_stub_collision.stl scale=1 1 1; collision mesh filename=meshes/jelly/jelly__deck_collision.stl scale=1 1 1
- link left_e1: mass 0.00207775 -> 3.75; geometry collision mesh filename=meshes/jelly/left_e1_collision.stl scale=1 1 1; visual mesh filename=meshes/jelly/left_e1_0.stl scale=1 1 1
- link left_e2: mass 0.000797087 -> 0.25; geometry collision mesh filename=meshes/jelly/left_e2_collision.stl scale=1 1 1; visual mesh filename=meshes/jelly/left_e2_0.stl scale=1 1 1
- link left_finger_1: mass None -> 0.04; geometry collision mesh filename=meshes/jelly/left_finger_1_collision.stl scale=1 1 1; visual mesh filename=meshes/jelly/left_finger_1_0.stl scale=1 1 1
- link left_finger_2: mass None -> 0.04; geometry collision mesh filename=meshes/jelly/left_finger_2_collision.stl scale=1 1 1; visual mesh filename=meshes/jelly/left_finger_2_0.stl scale=1 1 1
- link left_fingers: geometry 
- link left_gripper: mass 0.00042575 -> 0.25; geometry collision mesh filename=meshes/jelly/left_gripper_collision.stl scale=1 1 1; visual mesh filename=meshes/jelly/left_gripper_0.stl scale=1 1 1
- link left_s2: mass 0.00108759 -> 1.8; geometry collision mesh filename=meshes/jelly/left_s2_collision.stl scale=1 1 1; visual mesh filename=meshes/jelly/left_s2_0.stl scale=1 1 1
- link left_s3: mass 0.000265068 -> 1; geometry collision mesh filename=meshes/jelly/left_s3_collision.stl scale=1 1 1; visual mesh filename=meshes/jelly/left_s3_0.stl scale=1 1 1
- link left_w0: mass 0.0005018 -> 0.25; geometry collision mesh filename=meshes/jelly/left_w0_collision.stl scale=1 1 1; visual mesh filename=meshes/jelly/left_w0_0.stl scale=1 1 1
- link left_w1: mass 0.000330643 -> 0.65; geometry collision mesh filename=meshes/jelly/left_w1_collision.stl scale=1 1 1; visual mesh filename=meshes/jelly/left_w1_0.stl scale=1 1 1
- link left_w2: mass 4.33287e-05 -> 0.34; geometry collision mesh filename=meshes/jelly/left_w2_collision.stl scale=1 1 1; visual mesh filename=meshes/jelly/left_w2_0.stl scale=1 1 1
- link left_wrist_camera: mass None -> 0.08; geometry collision mesh filename=meshes/jelly/left_wrist_camera_collision.stl scale=1 1 1; visual mesh filename=meshes/jelly/left_wrist_camera_0.stl scale=1 1 1
- link lift_plate: mass None -> 1; geometry collision mesh filename=meshes/jelly/lift_plate_collision.stl scale=1 1 1
- link lift_stage: mass None -> 3; geometry collision mesh filename=meshes/jelly/lift_stage__column_mid_collision.stl scale=1 1 1; visual mesh filename=meshes/jelly/lift_stage_0.stl scale=1 1 1
- link right_e1: mass 0.00207775 -> 3.75; geometry collision mesh filename=meshes/jelly/right_e1_collision.stl scale=1 1 1; visual mesh filename=meshes/jelly/right_e1_0.stl scale=1 1 1
- link right_e2: mass 0.000797087 -> 0.25; geometry collision mesh filename=meshes/jelly/right_e2_collision.stl scale=1 1 1; visual mesh filename=meshes/jelly/right_e2_0.stl scale=1 1 1
- link right_finger_1: mass None -> 0.04; geometry collision mesh filename=meshes/jelly/right_finger_1_collision.stl scale=1 1 1; visual mesh filename=meshes/jelly/right_finger_1_0.stl scale=1 1 1
- link right_finger_2: mass None -> 0.04; geometry collision mesh filename=meshes/jelly/right_finger_2_collision.stl scale=1 1 1; visual mesh filename=meshes/jelly/right_finger_2_0.stl scale=1 1 1
- link right_fingers: geometry 
- link right_gripper: mass 0.00042575 -> 0.25; geometry collision mesh filename=meshes/jelly/right_gripper_collision.stl scale=1 1 1; visual mesh filename=meshes/jelly/right_gripper_0.stl scale=1 1 1
- link right_s2: mass 0.00108759 -> 1.8; geometry collision mesh filename=meshes/jelly/right_s2_collision.stl scale=1 1 1; visual mesh filename=meshes/jelly/right_s2_0.stl scale=1 1 1
- link right_s3: mass 0.000265068 -> 1; geometry collision mesh filename=meshes/jelly/right_s3_collision.stl scale=1 1 1; visual mesh filename=meshes/jelly/right_s3_0.stl scale=1 1 1
- link right_w0: mass 0.0005018 -> 0.25; geometry collision mesh filename=meshes/jelly/right_w0_collision.stl scale=1 1 1; visual mesh filename=meshes/jelly/right_w0_0.stl scale=1 1 1
- link right_w1: mass 0.000330643 -> 0.65; geometry collision mesh filename=meshes/jelly/right_w1_collision.stl scale=1 1 1; visual mesh filename=meshes/jelly/right_w1_0.stl scale=1 1 1
- link right_w2: mass 4.33287e-05 -> 0.34; geometry collision mesh filename=meshes/jelly/right_w2_collision.stl scale=1 1 1; visual mesh filename=meshes/jelly/right_w2_0.stl scale=1 1 1
- link right_wrist_camera: mass None -> 0.08; geometry collision mesh filename=meshes/jelly/right_wrist_camera_collision.stl scale=1 1 1; visual mesh filename=meshes/jelly/right_wrist_camera_0.stl scale=1 1 1
- link s1: mass 0.003744 -> 3; geometry collision mesh filename=meshes/jelly/s1_collision.stl scale=1 1 1; visual mesh filename=meshes/jelly/s1_0.stl scale=1 1 1
- link wheel_1_link: mass None -> 1; geometry collision mesh filename=meshes/jelly/wheel_1_link_collision.stl scale=1 1 1; visual mesh filename=meshes/jelly/wheel_1_link_0.stl scale=1 1 1
- link wheel_2_link: mass None -> 1; geometry collision mesh filename=meshes/jelly/wheel_2_link_collision.stl scale=1 1 1; visual mesh filename=meshes/jelly/wheel_2_link_0.stl scale=1 1 1
- link wheel_3_link: mass None -> 1; geometry collision mesh filename=meshes/jelly/wheel_3_link_collision.stl scale=1 1 1; visual mesh filename=meshes/jelly/wheel_3_link_0.stl scale=1 1 1
- link wheel_4_link: mass None -> 1; geometry collision mesh filename=meshes/jelly/wheel_4_link_collision.stl scale=1 1 1; visual mesh filename=meshes/jelly/wheel_4_link_0.stl scale=1 1 1
Joints:
- removed joint jelly_0
- removed joint left_finger_1_0
- removed joint left_finger_2_0
- removed joint lift_stage_0
- removed joint right_finger_1_0
- removed joint right_finger_2_0
- removed joint wheel_1_link_0
- removed joint wheel_2_link_0
- removed joint wheel_3_link_0
- removed joint wheel_4_link_0
- added joint base_x: type prismatic, parent world, child base_x_link, origin xyz=-0.112228 5.24549e-06 -0.46944 rpy=0 0 0, axis 1 0 0, limit lower=-10 upper=10 effort=1000 velocity=1
- added joint base_y: type prismatic, parent base_x_link, child base_y_link, origin xyz=0 0 0 rpy=0 0 0, axis 0 1 0, limit lower=-10 upper=10 effort=1000 velocity=1
- added joint base_yaw: type revolute, parent base_y_link, child jelly, origin xyz=0 0 0 rpy=0 0 0, axis 0 0 1, limit lower=-6.28319 upper=6.28319 effort=1000 velocity=1
- added joint deck_0_0: type fixed, parent jelly, child deck_0, origin xyz=0 0 0 rpy=0 0 0
- added joint deck_1_0: type fixed, parent jelly, child deck_1, origin xyz=0 0 0 rpy=0 0 0
- added joint deck_2_0: type fixed, parent jelly, child deck_2, origin xyz=0 0 0 rpy=0 0 0
- added joint left_finger_1_joint: type prismatic, parent left_gripper, child left_finger_1, origin xyz=0.0125619 0.0340885 -0.0542893 rpy=1.57079 -2.65359e-06 -3.14159, axis 1 0 0, limit lower=-2.15395e-13 upper=0.058804 effort=50 velocity=0.1
- added joint left_finger_2_joint: type prismatic, parent left_gripper, child left_finger_2, origin xyz=-0.0125578 -0.0324116 -0.0542893 rpy=1.5708 -3.76379e-12 4.69282e-06, axis 1 0 0, limit lower=-2.15451e-13 upper=0.058804 effort=50 velocity=0.1, mimic joint=left_finger_1_joint multiplier=1 offset=0
- added joint lift: type prismatic, parent jelly, child lift_stage, origin xyz=0 0 0 rpy=0 0 0, axis 0 0 -1, limit lower=0 upper=0.34 effort=1000 velocity=0.03
- added joint lift_2: type prismatic, parent lift_stage, child root, origin xyz=0.112228 -5.24549e-06 0.46944 rpy=0 0 0, axis 0 0 -1, limit lower=0 upper=0.34 effort=1000 velocity=0.03, mimic joint=lift multiplier=1 offset=0
- added joint right_finger_1_joint: type prismatic, parent right_gripper, child right_finger_1, origin xyz=0.0125624 0.0340829 -0.0542888 rpy=1.5708 -1e-05 -3.14159, axis 1 0 0, limit lower=-2.15395e-13 upper=0.058804 effort=50 velocity=0.1
- added joint right_finger_2_joint: type prismatic, parent right_gripper, child right_finger_2, origin xyz=-0.0125574 -0.0324172 -0.0542887 rpy=1.5708 7.34641e-06 3.26795e-06, axis 1 0 0, limit lower=-2.15451e-13 upper=0.058804 effort=50 velocity=0.1, mimic joint=right_finger_1_joint multiplier=1 offset=0
- added joint wheel_1: type continuous, parent jelly, child wheel_1_link, origin xyz=0.215834 0.215832 0.06335 rpy=3.14159 0 0, axis -0.707107 0.707107 0, limit effort=20 velocity=30
- added joint wheel_2: type continuous, parent jelly, child wheel_2_link, origin xyz=0.215832 -0.215834 0.06335 rpy=0 0 -5.30718e-06, axis -0.707107 0.707107 0, limit effort=20 velocity=30
- added joint wheel_3: type continuous, parent jelly, child wheel_3_link, origin xyz=-0.215832 0.215834 0.06335 rpy=0 0 0, axis 0.707107 -0.707107 0, limit effort=20 velocity=30
- added joint wheel_4: type continuous, parent jelly, child wheel_4_link, origin xyz=-0.215834 -0.215832 0.06335 rpy=3.14159 0 0, axis 0.707107 -0.707107 0, limit effort=20 velocity=30
- joint floor_0: parent root -> world

File: almond_axol/kinematics/urdf/axol_jelly_parcel.urdf (robot description, URDF)
Before this commit: robot assembly, 34 links, 33 joints
Links:
- added link base_x_link, mass 0.01
- added link base_y_link, mass 0.01
- added link deck_0
- added link deck_1
- added link deck_2
- added link world
- link base: mass 0.02496 -> 4; geometry collision mesh filename=meshes/jelly/base__column_top_collision.stl scale=1 1 1; visual mesh filename=meshes/jelly/base_0.stl scale=1 1 1
- link head: mass None -> 0.3; geometry collision mesh filename=meshes/jelly_parcel/head_collision.stl scale=1 1 1; visual mesh filename=meshes/jelly/head_1.stl scale=1 1 1
- link jelly: mass None -> 40; geometry collision mesh filename=meshes/jelly/jelly__column_stub_collision.stl scale=1 1 1; collision mesh filename=meshes/jelly/jelly__deck_collision.stl scale=1 1 1
- link left_e1: mass 0.00207775 -> 3.75; geometry collision mesh filename=meshes/jelly/left_e1_collision.stl scale=1 1 1; visual mesh filename=meshes/jelly/left_e1_0.stl scale=1 1 1
- link left_e2: mass 0.000797087 -> 0.25; geometry collision mesh filename=meshes/jelly/left_e2_collision.stl scale=1 1 1; visual mesh filename=meshes/jelly/left_e2_0.stl scale=1 1 1
- link left_fingers: geometry 
- link left_gripper: mass 0.00042575 -> 0.3; geometry collision mesh filename=meshes/jelly_parcel/left_gripper_collision.stl scale=1 1 1; visual mesh filename=meshes/jelly_parcel/left_gripper_0.stl scale=1 1 1
- link left_plate: mass None -> 0.08; geometry collision mesh filename=meshes/jelly_parcel/left_plate_collision.stl scale=1 1 1; visual mesh filename=meshes/jelly_parcel/left_plate_0.stl scale=1 1 1
- link left_s2: mass 0.00108759 -> 1.8; geometry collision mesh filename=meshes/jelly/left_s2_collision.stl scale=1 1 1; visual mesh filename=meshes/jelly/left_s2_0.stl scale=1 1 1
- link left_s3: mass 0.000265068 -> 1; geometry collision mesh filename=meshes/jelly/left_s3_collision.stl scale=1 1 1; visual mesh filename=meshes/jelly/left_s3_0.stl scale=1 1 1
- link left_w0: mass 0.0005018 -> 0.25; geometry collision mesh filename=meshes/jelly/left_w0_collision.stl scale=1 1 1; visual mesh filename=meshes/jelly/left_w0_0.stl scale=1 1 1
- link left_w1: mass 0.000330643 -> 0.65; geometry collision mesh filename=meshes/jelly/left_w1_collision.stl scale=1 1 1; visual mesh filename=meshes/jelly/left_w1_0.stl scale=1 1 1
- link left_w2: mass 4.33287e-05 -> 0.37; geometry collision mesh filename=meshes/jelly_parcel/left_w2_collision.stl scale=1 1 1; visual mesh filename=meshes/jelly_parcel/left_w2_0.stl scale=1 1 1
- link lift_plate: mass None -> 1; geometry collision mesh filename=meshes/jelly/lift_plate_collision.stl scale=1 1 1
- link lift_stage: mass None -> 3; geometry collision mesh filename=meshes/jelly/lift_stage__column_mid_collision.stl scale=1 1 1; visual mesh filename=meshes/jelly/lift_stage_0.stl scale=1 1 1
- link right_e1: mass 0.00207775 -> 3.75; geometry collision mesh filename=meshes/jelly/right_e1_collision.stl scale=1 1 1; visual mesh filename=meshes/jelly/right_e1_0.stl scale=1 1 1
- link right_e2: mass 0.000797087 -> 0.25; geometry collision mesh filename=meshes/jelly/right_e2_collision.stl scale=1 1 1; visual mesh filename=meshes/jelly/right_e2_0.stl scale=1 1 1
- link right_fingers: geometry 
- link right_gripper: mass 0.00042575 -> 0.3; geometry collision mesh filename=meshes/jelly_parcel/right_gripper_collision.stl scale=1 1 1; visual mesh filename=meshes/jelly_parcel/right_gripper_0.stl scale=1 1 1
- link right_plate: mass None -> 0.08; geometry collision mesh filename=meshes/jelly_parcel/right_plate_collision.stl scale=1 1 1; visual mesh filename=meshes/jelly_parcel/right_plate_0.stl scale=1 1 1
- link right_s2: mass 0.00108759 -> 1.8; geometry collision mesh filename=meshes/jelly/right_s2_collision.stl scale=1 1 1; visual mesh filename=meshes/jelly/right_s2_0.stl scale=1 1 1
- link right_s3: mass 0.000265068 -> 1; geometry collision mesh filename=meshes/jelly/right_s3_collision.stl scale=1 1 1; visual mesh filename=meshes/jelly/right_s3_0.stl scale=1 1 1
- link right_w0: mass 0.0005018 -> 0.25; geometry collision mesh filename=meshes/jelly/right_w0_collision.stl scale=1 1 1; visual mesh filename=meshes/jelly/right_w0_0.stl scale=1 1 1
- link right_w1: mass 0.000330643 -> 0.65; geometry collision mesh filename=meshes/jelly/right_w1_collision.stl scale=1 1 1; visual mesh filename=meshes/jelly/right_w1_0.stl scale=1 1 1
- link right_w2: mass 4.33287e-05 -> 0.37; geometry collision mesh filename=meshes/jelly_parcel/right_w2_collision.stl scale=1 1 1; visual mesh filename=meshes/jelly_parcel/right_w2_0.stl scale=1 1 1
- link s1: mass 0.003744 -> 3; geometry collision mesh filename=meshes/jelly/s1_collision.stl scale=1 1 1; visual mesh filename=meshes/jelly/s1_0.stl scale=1 1 1
- link wheel_1_link: mass None -> 1; geometry collision mesh filename=meshes/jelly/wheel_1_link_collision.stl scale=1 1 1; visual mesh filename=meshes/jelly/wheel_1_link_0.stl scale=1 1 1
- link wheel_2_link: mass None -> 1; geometry collision mesh filename=meshes/jelly_parcel/wheel_2_link_collision.stl scale=1 1 1; visual mesh filename=meshes/jelly_parcel/wheel_2_link_0.stl scale=1 1 1
- link wheel_3_link: mass None -> 1; geometry collision mesh filename=meshes/jelly_parcel/wheel_3_link_collision.stl scale=1 1 1; visual mesh filename=meshes/jelly_parcel/wheel_3_link_0.stl scale=1 1 1
- link wheel_4_link: mass None -> 1; geometry collision mesh filename=meshes/jelly/wheel_4_link_collision.stl scale=1 1 1; visual mesh filename=meshes/jelly/wheel_4_link_0.stl scale=1 1 1
Joints:
- removed joint jelly_0
- removed joint left_plate_0
- removed joint lift_stage_0
- removed joint right_plate_0
- removed joint wheel_1_link_0
- removed joint wheel_2_link_0
- removed joint wheel_3_link_0
- removed joint wheel_4_link_0
- added joint base_x: type prismatic, parent world, child base_x_link, origin xyz=-0.112228 5.36873e-06 -0.46944 rpy=0 0 0, axis 1 0 0, limit lower=-10 upper=10 effort=1000 velocity=1
- added joint base_y: type prismatic, parent base_x_link, child base_y_link, origin xyz=0 0 0 rpy=0 0 0, axis 0 1 0, limit lower=-10 upper=10 effort=1000 velocity=1
- added joint base_yaw: type revolute, parent base_y_link, child jelly, origin xyz=0 0 0 rpy=0 0 0, axis 0 0 1, limit lower=-6.28319 upper=6.28319 effort=1000 velocity=1
- added joint deck_0_0: type fixed, parent jelly, child deck_0, origin xyz=0 0 0 rpy=0 0 0
- added joint deck_1_0: type fixed, parent jelly, child deck_1, origin xyz=0 0 0 rpy=0 0 0
- added joint deck_2_0: type fixed, parent jelly, child deck_2, origin xyz=0 0 0 rpy=0 0 0
- added joint left_plate_joint: type revolute, parent left_gripper, child left_plate, origin xyz=-0.0114984 0.0235875 -0.0399892 rpy=3.14158 1.57079 1.57079, axis 0 0 1, limit lower=-3.14159 upper=0 effort=5 velocity=3
- added joint lift: type prismatic, parent jelly, child lift_stage, origin xyz=0 0 0 rpy=0 0 0, axis 0 0 -1, limit lower=0 upper=0.34 effort=1000 velocity=0.03
- added joint lift_2: type prismatic, parent lift_stage, child root, origin xyz=0.112228 -5.36873e-06 0.46944 rpy=0 0 0, axis 0 0 -1, limit lower=0 upper=0.34 effort=1000 velocity=0.03, mimic joint=lift multiplier=1 offset=0
- added joint right_plate_joint: type revolute, parent right_gripper, child right_plate, origin xyz=0.0115022 0.0235838 -0.0399889 rpy=-1.10715 1.57079 -2.67794, axis 0 0 1, limit lower=0 upper=3.14159 effort=5 velocity=3
- added joint wheel_1: type continuous, parent jelly, child wheel_1_link, origin xyz=0.215834 0.215832 0.06335 rpy=3.14159 0 0, axis -0.707107 0.707107 0, limit effort=20 velocity=30
- added joint wheel_2: type continuous, parent jelly, child wheel_2_link, origin xyz=-0.215834 -0.215832 0.06335 rpy=3.14159 0 0, axis -0.707107 0.707107 0, limit effort=20 velocity=30
- added joint wheel_3: type continuous, parent jelly, child wheel_3_link, origin xyz=0.215832 -0.215834 0.06335 rpy=0 0 -5.30718e-06, axis 0.707107 -0.707107 0, limit effort=20 velocity=30
- added joint wheel_4: type continuous, parent jelly, child wheel_4_link, origin xyz=-0.215832 0.215834 0.06335 rpy=0 0 0, axis 0.707107 -0.707107 0, limit effort=20 velocity=30
- joint floor_0: parent root -> world
