Commit message: One URDF per Axol version: IK, viewers and simulators share one full model
The generated versions are now one file each — axol_standalone,
axol_ox_cart, axol_owl, axol_jelly, and axol_jelly_parcel for the parcel
gripper — next to the legacy axol.urdf. The Jelly arm-IK, whole-body and
sim files are merged into axol_jelly.urdf (and likewise for parcel).

Each file is the full robot: every moving part a joint (the Jelly base in
the plane and its two-stage lift, the Ox cart's lift, fingers or parcel
plate, wheels), AxolConfig's arm masses with estimates elsewhere, friction
and drive gains, per-part contact hulls in <collision>, and relative mesh
paths. With every body joint at zero the torso is the world origin, so IK
frames and recorded poses are unchanged. IK loads it through
kinematics.model.ik_urdf, which freezes the joints it does not solve (arm
IK: all but the arms; whole-body IK: plus base and lift) and collides the
capsule-friendly <ik_collision> pieces instead.

Jelly arm IK now collides the lift column per section (the whole-body
split) rather than one hull over all three: 96 pairs instead of 64, ~0.7 ms
more per solve. The full models' own masses weigh the arms exactly as
gravity compensation's tuned model (checked in MuJoCo with fusestatic off).

The generator is renamed scripts/build_urdfs.py and models each body's IK
and physics collision sets, lift and masses on its Body.

Co-Authored-By: Claude Opus 5.5 <noreply@anthropic.com>

File: almond_axol/kinematics/urdf/axol_owl.urdf (robot description, URDF)
Before this commit: robot assembly, 38 links, 37 joints
Links:
- link base: mass 0.02496 -> 3; geometry collision mesh filename=meshes/owl/base__foot_collision.stl scale=1 1 1; collision mesh filename=meshes/owl/base_collision.stl scale=1 1 1
- link foot_0: geometry 
- link foot_1: geometry 
- link foot_2: geometry 
- link foot_3: geometry 
- link foot_4: geometry 
- link foot_5: geometry 
- link head: mass None -> 0.3; geometry collision mesh filename=meshes/jelly/head_collision.stl scale=1 1 1; visual mesh filename=meshes/jelly/head_0.stl scale=1 1 1
- link left_e1: mass 0.00207775 -> 3.75; geometry collision mesh filename=meshes/jelly/left_e1_collision.stl scale=1 1 1; visual mesh filename=meshes/jelly/left_e1_0.stl scale=1 1 1
- link left_e2: mass 0.000797087 -> 0.25; geometry collision mesh filename=meshes/jelly/left_e2_collision.stl scale=1 1 1; visual mesh filename=meshes/jelly/left_e2_0.stl scale=1 1 1
- link left_finger_1: mass None -> 0.04; geometry collision mesh filename=meshes/standalone/left_finger_1_collision.stl scale=1 1 1; visual mesh filename=meshes/jelly/left_finger_1_0.stl scale=1 1 1
- link left_finger_2: mass None -> 0.04; geometry collision mesh filename=meshes/standalone/left_finger_2_collision.stl scale=1 1 1; visual mesh filename=meshes/jelly/left_finger_2_0.stl scale=1 1 1
- link left_fingers: geometry 
- link left_gripper: mass 0.00042575 -> 0.25; geometry collision mesh filename=meshes/jelly/left_gripper_collision.stl scale=1 1 1; visual mesh filename=meshes/jelly/left_gripper_0.stl scale=1 1 1
- link left_s2: mass 0.00108759 -> 1.8; geometry collision mesh filename=meshes/jelly/left_s2_collision.stl scale=1 1 1; visual mesh filename=meshes/jelly/left_s2_0.stl scale=1 1 1
- link left_s3: mass 0.000265068 -> 1; geometry collision mesh filename=meshes/jelly/left_s3_collision.stl scale=1 1 1; visual mesh filename=meshes/jelly/left_s3_0.stl scale=1 1 1
- link left_w0: mass 0.0005018 -> 0.25; geometry collision mesh filename=meshes/jelly/left_w0_collision.stl scale=1 1 1; visual mesh filename=meshes/jelly/left_w0_0.stl scale=1 1 1
- link left_w1: mass 0.000330643 -> 0.65; geometry collision mesh filename=meshes/jelly/left_w1_collision.stl scale=1 1 1; visual mesh filename=meshes/jelly/left_w1_0.stl scale=1 1 1
- link left_w2: mass 4.33287e-05 -> 0.34; geometry collision mesh filename=meshes/standalone/left_w2_collision.stl scale=1 1 1; visual mesh filename=meshes/standalone/left_w2_0.stl scale=1 1 1
- link left_wrist_camera: mass None -> 0.08; geometry collision mesh filename=meshes/jelly/left_wrist_camera_collision.stl scale=1 1 1; visual mesh filename=meshes/jelly/left_wrist_camera_0.stl scale=1 1 1
- link right_e1: mass 0.00207775 -> 3.75; geometry collision mesh filename=meshes/jelly/right_e1_collision.stl scale=1 1 1; visual mesh filename=meshes/jelly/right_e1_0.stl scale=1 1 1
- link right_e2: mass 0.000797087 -> 0.25; geometry collision mesh filename=meshes/jelly/right_e2_collision.stl scale=1 1 1; visual mesh filename=meshes/jelly/right_e2_0.stl scale=1 1 1
- link right_finger_1: mass None -> 0.04; geometry collision mesh filename=meshes/standalone/right_finger_1_collision.stl scale=1 1 1; visual mesh filename=meshes/jelly/right_finger_1_0.stl scale=1 1 1
- link right_finger_2: mass None -> 0.04; geometry collision mesh filename=meshes/standalone/right_finger_2_collision.stl scale=1 1 1; visual mesh filename=meshes/jelly/right_finger_2_0.stl scale=1 1 1
- link right_fingers: geometry 
- link right_gripper: mass 0.00042575 -> 0.25; geometry collision mesh filename=meshes/jelly/right_gripper_collision.stl scale=1 1 1; visual mesh filename=meshes/jelly/right_gripper_0.stl scale=1 1 1
- link right_s2: mass 0.00108759 -> 1.8; geometry collision mesh filename=meshes/jelly/right_s2_collision.stl scale=1 1 1; visual mesh filename=meshes/jelly/right_s2_0.stl scale=1 1 1
- link right_s3: mass 0.000265068 -> 1; geometry collision mesh filename=meshes/jelly/right_s3_collision.stl scale=1 1 1; visual mesh filename=meshes/jelly/right_s3_0.stl scale=1 1 1
- link right_w0: mass 0.0005018 -> 0.25; geometry collision mesh filename=meshes/jelly/right_w0_collision.stl scale=1 1 1; visual mesh filename=meshes/jelly/right_w0_0.stl scale=1 1 1
- link right_w1: mass 0.000330643 -> 0.65; geometry collision mesh filename=meshes/jelly/right_w1_collision.stl scale=1 1 1; visual mesh filename=meshes/jelly/right_w1_0.stl scale=1 1 1
- link right_w2: mass 4.33287e-05 -> 0.34; geometry collision mesh filename=meshes/standalone/right_w2_collision.stl scale=1 1 1; visual mesh filename=meshes/standalone/right_w2_0.stl scale=1 1 1
- link right_wrist_camera: mass None -> 0.08; geometry collision mesh filename=meshes/jelly/right_wrist_camera_collision.stl scale=1 1 1; visual mesh filename=meshes/jelly/right_wrist_camera_0.stl scale=1 1 1
- link s1: mass 0.003744 -> 3; geometry collision mesh filename=meshes/jelly/s1_collision.stl scale=1 1 1; visual mesh filename=meshes/jelly/s1_0.stl scale=1 1 1
Joints:
- removed joint left_finger_1_0
- removed joint left_finger_2_0
- removed joint right_finger_1_0
- removed joint right_finger_2_0
- added joint left_finger_1_joint: type prismatic, parent left_gripper, child left_finger_1, origin xyz=0.0341019 0.0225863 -0.0575393 rpy=1.57079 -2.65359e-06 3.14159, axis -1 0 0, limit lower=-0.0330428 upper=0.0109572 effort=50 velocity=0.1
- added joint left_finger_2_joint: type prismatic, parent left_gripper, child left_finger_2, origin xyz=-0.0341078 -0.0224134 -0.0575393 rpy=1.5708 -3.75488e-12 -5.30718e-06, axis -1 0 0, limit lower=-0.0330428 upper=0.0109572 effort=50 velocity=0.1, mimic joint=left_finger_1_joint multiplier=1 offset=0
- added joint right_finger_1_joint: type prismatic, parent right_gripper, child right_finger_1, origin xyz=0.0341024 0.0225842 -0.0575391 rpy=1.5708 -9.99996e-06 3.14158, axis -1 0 0, limit lower=-0.0330428 upper=0.0109572 effort=50 velocity=0.1
- added joint right_finger_2_joint: type prismatic, parent right_gripper, child right_finger_2, origin xyz=-0.0341076 -0.022415 -0.0575384 rpy=1.57079 7.34637e-06 -1.20392e-05, axis -1 0 0, limit lower=-0.0330428 upper=0.0109572 effort=50 velocity=0.1, mimic joint=right_finger_1_joint multiplier=1 offset=0

File: almond_axol/kinematics/urdf/axol_ox_cart.urdf (robot description, URDF)
Before this commit: robot assembly, 34 links, 33 joints
Links:
- added link world
- link base: mass 0.02496 -> 6; geometry collision mesh filename=meshes/ox_cart/base_collision.stl scale=1 1 1; visual mesh filename=meshes/ox_cart/base_0.stl scale=1 1 1
- link cart: mass None -> 30; geometry collision mesh filename=meshes/ox_cart/cart__cart_frame_collision.stl scale=1 1 1; collision mesh filename=meshes/ox_cart/cart__column_stub_collision.stl scale=1 1 1
- link head: mass None -> 0.3; geometry collision mesh filename=meshes/jelly/head_collision.stl scale=1 1 1; visual mesh filename=meshes/jelly/head_0.stl scale=1 1 1
- link left_e1: mass 0.00207775 -> 3.75; geometry collision mesh filename=meshes/jelly/left_e1_collision.stl scale=1 1 1; visual mesh filename=meshes/jelly/left_e1_0.stl scale=1 1 1
- link left_e2: mass 0.000797087 -> 0.25; geometry collision mesh filename=meshes/jelly/left_e2_collision.stl scale=1 1 1; visual mesh filename=meshes/jelly/left_e2_0.stl scale=1 1 1
- link left_finger_1: mass None -> 0.04; geometry collision mesh filename=meshes/standalone/left_finger_1_collision.stl scale=1 1 1; visual mesh filename=meshes/jelly/left_finger_1_0.stl scale=1 1 1
- link left_finger_2: mass None -> 0.04; geometry collision mesh filename=meshes/standalone/left_finger_2_collision.stl scale=1 1 1; visual mesh filename=meshes/jelly/left_finger_2_0.stl scale=1 1 1
- link left_fingers: geometry 
- link left_gripper: mass 0.00042575 -> 0.25; geometry collision mesh filename=meshes/jelly/left_gripper_collision.stl scale=1 1 1; visual mesh filename=meshes/jelly/left_gripper_0.stl scale=1 1 1
- link left_s2: mass 0.00108759 -> 1.8; geometry collision mesh filename=meshes/jelly/left_s2_collision.stl scale=1 1 1; visual mesh filename=meshes/jelly/left_s2_0.stl scale=1 1 1
- link left_s3: mass 0.000265068 -> 1; geometry collision mesh filename=meshes/jelly/left_s3_collision.stl scale=1 1 1; visual mesh filename=meshes/jelly/left_s3_0.stl scale=1 1 1
- link left_w0: mass 0.0005018 -> 0.25; geometry collision mesh filename=meshes/jelly/left_w0_collision.stl scale=1 1 1; visual mesh filename=meshes/jelly/left_w0_0.stl scale=1 1 1
- link left_w1: mass 0.000330643 -> 0.65; geometry collision mesh filename=meshes/jelly/left_w1_collision.stl scale=1 1 1; visual mesh filename=meshes/jelly/left_w1_0.stl scale=1 1 1
- link left_w2: mass 4.33287e-05 -> 0.34; geometry collision mesh filename=meshes/standalone/left_w2_collision.stl scale=1 1 1; visual mesh filename=meshes/standalone/left_w2_0.stl scale=1 1 1
- link left_wrist_camera: mass None -> 0.08; geometry collision mesh filename=meshes/jelly/left_wrist_camera_collision.stl scale=1 1 1; visual mesh filename=meshes/jelly/left_wrist_camera_0.stl scale=1 1 1
- link right_e1: mass 0.00207775 -> 3.75; geometry collision mesh filename=meshes/jelly/right_e1_collision.stl scale=1 1 1; visual mesh filename=meshes/jelly/right_e1_0.stl scale=1 1 1
- link right_e2: mass 0.000797087 -> 0.25; geometry collision mesh filename=meshes/jelly/right_e2_collision.stl scale=1 1 1; visual mesh filename=meshes/jelly/right_e2_0.stl scale=1 1 1
- link right_finger_1: mass None -> 0.04; geometry collision mesh filename=meshes/standalone/right_finger_1_collision.stl scale=1 1 1; visual mesh filename=meshes/jelly/right_finger_1_0.stl scale=1 1 1
- link right_finger_2: mass None -> 0.04; geometry collision mesh filename=meshes/standalone/right_finger_2_collision.stl scale=1 1 1; visual mesh filename=meshes/jelly/right_finger_2_0.stl scale=1 1 1
- link right_fingers: geometry 
- link right_gripper: mass 0.00042575 -> 0.25; geometry collision mesh filename=meshes/jelly/right_gripper_collision.stl scale=1 1 1; visual mesh filename=meshes/jelly/right_gripper_0.stl scale=1 1 1
- link right_s2: mass 0.00108759 -> 1.8; geometry collision mesh filename=meshes/jelly/right_s2_collision.stl scale=1 1 1; visual mesh filename=meshes/jelly/right_s2_0.stl scale=1 1 1
- link right_s3: mass 0.000265068 -> 1; geometry collision mesh filename=meshes/jelly/right_s3_collision.stl scale=1 1 1; visual mesh filename=meshes/jelly/right_s3_0.stl scale=1 1 1
- link right_w0: mass 0.0005018 -> 0.25; geometry collision mesh filename=meshes/jelly/right_w0_collision.stl scale=1 1 1; visual mesh filename=meshes/jelly/right_w0_0.stl scale=1 1 1
- link right_w1: mass 0.000330643 -> 0.65; geometry collision mesh filename=meshes/jelly/right_w1_collision.stl scale=1 1 1; visual mesh filename=meshes/jelly/right_w1_0.stl scale=1 1 1
- link right_w2: mass 4.33287e-05 -> 0.34; geometry collision mesh filename=meshes/standalone/right_w2_collision.stl scale=1 1 1; visual mesh filename=meshes/standalone/right_w2_0.stl scale=1 1 1
- link right_wrist_camera: mass None -> 0.08; geometry collision mesh filename=meshes/jelly/right_wrist_camera_collision.stl scale=1 1 1; visual mesh filename=meshes/jelly/right_wrist_camera_0.stl scale=1 1 1
- link s1: mass 0.003744 -> 3; geometry collision mesh filename=meshes/jelly/s1_collision.stl scale=1 1 1; visual mesh filename=meshes/jelly/s1_0.stl scale=1 1 1
Joints:
- removed joint left_finger_1_0
- removed joint left_finger_2_0
- removed joint right_finger_1_0
- removed joint right_finger_2_0
- added joint left_finger_1_joint: type prismatic, parent left_gripper, child left_finger_1, origin xyz=0.0450634 0.0225889 -0.0575393 rpy=1.57079 -2.65357e-06 -3.14158, axis -1 0 0, limit lower=-0.044 upper=-2.77556e-17 effort=50 velocity=0.1
- added joint left_finger_2_joint: type prismatic, parent left_gripper, child left_finger_2, origin xyz=-0.04506 -0.022412 -0.0575393 rpy=1.5708 -2.31733e-11 1e-05, axis -1 0 0, limit lower=-0.044 upper=-5.55112e-17 effort=50 velocity=0.1, mimic joint=left_finger_1_joint multiplier=1 offset=0
- added joint lift: type prismatic, parent cart, child root, origin xyz=0.100357 -4.23699e-06 0.31251 rpy=0 0 0, axis 0 0 -1, limit lower=0 upper=0.4572 effort=1000 velocity=0.03
- added joint right_finger_1_joint: type prismatic, parent right_gripper, child right_finger_1, origin xyz=0.0450638 0.022583 -0.0575391 rpy=1.57079 -1e-05 -3.14159, axis -1 0 0, limit lower=-0.044 upper=-2.77556e-17 effort=50 velocity=0.1
- added joint right_finger_2_joint: type prismatic, parent right_gripper, child right_finger_2, origin xyz=-0.0450598 -0.0224173 -0.0575384 rpy=1.5708 7.34641e-06 3.26795e-06, axis -1 0 0, limit lower=-0.044 upper=-5.55112e-17 effort=50 velocity=0.1, mimic joint=right_finger_1_joint multiplier=1 offset=0
- joint cart_0: parent root -> world
- joint floor_0: parent root -> world

File: almond_axol/kinematics/urdf/axol_standalone.urdf (robot description, URDF)
Before this commit: robot assembly, 32 links, 31 joints
Links:
- link base: mass 0.02496 -> None
- link head: mass None -> 0.3; geometry collision mesh filename=meshes/jelly/head_collision.stl scale=1 1 1; visual mesh filename=meshes/jelly/head_0.stl scale=1 1 1
- link left_e1: mass 0.00207775 -> 3.75; geometry collision mesh filename=meshes/jelly/left_e1_collision.stl scale=1 1 1; visual mesh filename=meshes/jelly/left_e1_0.stl scale=1 1 1
- link left_e2: mass 0.000797087 -> 0.25; geometry collision mesh filename=meshes/jelly/left_e2_collision.stl scale=1 1 1; visual mesh filename=meshes/jelly/left_e2_0.stl scale=1 1 1
- link left_finger_1: mass None -> 0.04; geometry collision mesh filename=meshes/standalone/left_finger_1_collision.stl scale=1 1 1; visual mesh filename=meshes/jelly/left_finger_1_0.stl scale=1 1 1
- link left_finger_2: mass None -> 0.04; geometry collision mesh filename=meshes/standalone/left_finger_2_collision.stl scale=1 1 1; visual mesh filename=meshes/jelly/left_finger_2_0.stl scale=1 1 1
- link left_fingers: geometry 
- link left_gripper: mass 0.00042575 -> 0.25; geometry collision mesh filename=meshes/jelly/left_gripper_collision.stl scale=1 1 1; visual mesh filename=meshes/jelly/left_gripper_0.stl scale=1 1 1
- link left_s2: mass 0.00108759 -> 1.8; geometry collision mesh filename=meshes/jelly/left_s2_collision.stl scale=1 1 1; visual mesh filename=meshes/jelly/left_s2_0.stl scale=1 1 1
- link left_s3: mass 0.000265068 -> 1; geometry collision mesh filename=meshes/jelly/left_s3_collision.stl scale=1 1 1; visual mesh filename=meshes/jelly/left_s3_0.stl scale=1 1 1
- link left_w0: mass 0.0005018 -> 0.25; geometry collision mesh filename=meshes/jelly/left_w0_collision.stl scale=1 1 1; visual mesh filename=meshes/jelly/left_w0_0.stl scale=1 1 1
- link left_w1: mass 0.000330643 -> 0.65; geometry collision mesh filename=meshes/jelly/left_w1_collision.stl scale=1 1 1; visual mesh filename=meshes/jelly/left_w1_0.stl scale=1 1 1
- link left_w2: mass 4.33287e-05 -> 0.34; geometry collision mesh filename=meshes/standalone/left_w2_collision.stl scale=1 1 1; visual mesh filename=meshes/standalone/left_w2_0.stl scale=1 1 1
- link left_wrist_camera: mass None -> 0.08; geometry collision mesh filename=meshes/jelly/left_wrist_camera_collision.stl scale=1 1 1; visual mesh filename=meshes/jelly/left_wrist_camera_0.stl scale=1 1 1
- link right_e1: mass 0.00207775 -> 3.75; geometry collision mesh filename=meshes/jelly/right_e1_collision.stl scale=1 1 1; visual mesh filename=meshes/jelly/right_e1_0.stl scale=1 1 1
- link right_e2: mass 0.000797087 -> 0.25; geometry collision mesh filename=meshes/jelly/right_e2_collision.stl scale=1 1 1; visual mesh filename=meshes/jelly/right_e2_0.stl scale=1 1 1
- link right_finger_1: mass None -> 0.04; geometry collision mesh filename=meshes/standalone/right_finger_1_collision.stl scale=1 1 1; visual mesh filename=meshes/jelly/right_finger_1_0.stl scale=1 1 1
- link right_finger_2: mass None -> 0.04; geometry collision mesh filename=meshes/standalone/right_finger_2_collision.stl scale=1 1 1; visual mesh filename=meshes/jelly/right_finger_2_0.stl scale=1 1 1
- link right_fingers: geometry 
- link right_gripper: mass 0.00042575 -> 0.25; geometry collision mesh filename=meshes/jelly/right_gripper_collision.stl scale=1 1 1; visual mesh filename=meshes/jelly/right_gripper_0.stl scale=1 1 1
- link right_s2: mass 0.00108759 -> 1.8; geometry collision mesh filename=meshes/jelly/right_s2_collision.stl scale=1 1 1; visual mesh filename=meshes/jelly/right_s2_0.stl scale=1 1 1
- link right_s3: mass 0.000265068 -> 1; geometry collision mesh filename=meshes/jelly/right_s3_collision.stl scale=1 1 1; visual mesh filename=meshes/jelly/right_s3_0.stl scale=1 1 1
- link right_w0: mass 0.0005018 -> 0.25; geometry collision mesh filename=meshes/jelly/right_w0_collision.stl scale=1 1 1; visual mesh filename=meshes/jelly/right_w0_0.stl scale=1 1 1
- link right_w1: mass 0.000330643 -> 0.65; geometry collision mesh filename=meshes/jelly/right_w1_collision.stl scale=1 1 1; visual mesh filename=meshes/jelly/right_w1_0.stl scale=1 1 1
- link right_w2: mass 4.33287e-05 -> 0.34; geometry collision mesh filename=meshes/standalone/right_w2_collision.stl scale=1 1 1; visual mesh filename=meshes/standalone/right_w2_0.stl scale=1 1 1
- link right_wrist_camera: mass None -> 0.08; geometry collision mesh filename=meshes/jelly/right_wrist_camera_collision.stl scale=1 1 1; visual mesh filename=meshes/jelly/right_wrist_camera_0.stl scale=1 1 1
- link s1: mass 0.003744 -> 3; geometry collision mesh filename=meshes/jelly/s1_collision.stl scale=1 1 1; visual mesh filename=meshes/jelly/s1_0.stl scale=1 1 1
Joints:
- removed joint left_finger_1_0
- removed joint left_finger_2_0
- removed joint right_finger_1_0
- removed joint right_finger_2_0
- added joint left_finger_1_joint: type prismatic, parent left_gripper, child left_finger_1, origin xyz=0.045059 0.0225889 -0.0575393 rpy=1.57079 -2.65357e-06 -3.14158, axis -1 0 0, limit lower=-0.044 upper=-2.91434e-15 effort=50 velocity=0.1
- added joint left_finger_2_joint: type prismatic, parent left_gripper, child left_finger_2, origin xyz=-0.0450644 -0.022412 -0.0575393 rpy=1.5708 -2.3256e-11 1e-05, axis -1 0 0, limit lower=-0.044 upper=-6.91114e-15 effort=50 velocity=0.1, mimic joint=left_finger_1_joint multiplier=1 offset=0
- added joint right_finger_1_joint: type prismatic, parent right_gripper, child right_finger_1, origin xyz=0.0450595 0.0225828 -0.0575391 rpy=1.57079 -9.99998e-06 3.14159, axis -1 0 0, limit lower=-0.044 upper=-2.91434e-15 effort=50 velocity=0.1
- added joint right_finger_2_joint: type prismatic, parent right_gripper, child right_finger_2, origin xyz=-0.0450644 -0.022417 -0.0575384 rpy=1.5708 7.34639e-06 -2.03923e-06, axis -1 0 0, limit lower=-0.044 upper=-6.91114e-15 effort=50 velocity=0.1, mimic joint=right_finger_1_joint multiplier=1 offset=0

Commit message: Move whole-body IK out of this PR
Whole-body IK (solving the Jelly base and lift with the arms, sim only)
moves to its own PR, stacked on this one. Removed here: the
kinematics.whole_body switch and its body_* / *_max_delta tuning, the
solver's body joints, per-joint step budgets and moving shoulder centres,
BODY_JOINTS and the whole-body torso links, the Sim viewer's body joints,
the teleop body sink and the panel setting, and the Jelly deck's IK
collision strips.

The Jelly URDF keeps its base_x / base_y / base_yaw and lift joints for
physics simulators; IK now always freezes every joint but the arms'.

Co-Authored-By: Claude Opus 5.5 <noreply@anthropic.com>

File: almond_axol/kinematics/urdf/axol_jelly.urdf (robot description, URDF)
Before this commit: robot assembly, 46 links, 45 joints
Links:
- removed link deck_0
- removed link deck_1
- removed link deck_2
Joints:
- removed joint deck_0_0
- removed joint deck_1_0
- removed joint deck_2_0

File: almond_axol/kinematics/urdf/axol_jelly_parcel.urdf (robot description, URDF)
Before this commit: robot assembly, 40 links, 39 joints
Links:
- removed link deck_0
- removed link deck_1
- removed link deck_2
Joints:
- removed joint deck_0_0
- removed joint deck_1_0
- removed joint deck_2_0
