Commit message: Whole-body IK: solve the Jelly base and lift with the arms (sim only)
Stacked on axol-version-selector (#331), which ships the full Jelly model
with the base and lift as joints; this adds IK that moves them.

- kinematics.whole_body (control panel: Kinematics → Whole-body IK, sim
  only) adds base_x / base_y / base_yaw and the lift to the IK vector
  (BODY_JOINTS, after the 14 arm joints). The body holds still while both
  hands are within comfortable reach (body_reach_start / _band,
  body_hold_weight) and is damped once released (body_rest_weight), with
  its own per-solve step budgets (base_max_delta, base_yaw_max_delta,
  lift_max_delta); targets are not reach-clamped.
- The solver's shoulder centres and elbow-swivel geometry follow the base
  and lift; manipulability counts each arm's own joints only.
- IK collides the lift-column sections and the Jelly deck (as strips).
- axol teleop --sim drives the Sim viewer's base and lift; real hardware,
  absolute (Mantis) mode and data collection refuse the switch.

Co-Authored-By: Claude Opus 5.5 <noreply@anthropic.com>

File: almond_axol/kinematics/urdf/axol_jelly.urdf (robot description, URDF)
Before this commit: robot assembly, 43 links, 42 joints
Links:
- added link deck_0
- added link deck_1
- added link deck_2
Joints:
- added joint deck_0_0: type fixed, parent jelly, child deck_0, origin xyz=0 0 0 rpy=0 0 0
- added joint deck_1_0: type fixed, parent jelly, child deck_1, origin xyz=0 0 0 rpy=0 0 0
- added joint deck_2_0: type fixed, parent jelly, child deck_2, origin xyz=0 0 0 rpy=0 0 0

File: almond_axol/kinematics/urdf/axol_jelly_parcel.urdf (robot description, URDF)
Before this commit: robot assembly, 37 links, 36 joints
Links:
- added link deck_0
- added link deck_1
- added link deck_2
Joints:
- added joint deck_0_0: type fixed, parent jelly, child deck_0, origin xyz=0 0 0 rpy=0 0 0
- added joint deck_1_0: type fixed, parent jelly, child deck_1, origin xyz=0 0 0 rpy=0 0 0
- added joint deck_2_0: type fixed, parent jelly, child deck_2, origin xyz=0 0 0 rpy=0 0 0

Commit message: Ox cart stands on its casters; pick the robot model before the first run
- The floor link goes under the body's lowest point, not the export
  root: the Ox cart's root is its frame, 112 mm above the casters, so the
  cart sank through the viewers' ground plane. (Jelly moves 0.1 mm.)
- Until a robot model is saved (kinematics.mount), the control panel
  shows "Which Axol is this?" above Axol settings and lists it under
  "Before you can start" for Axol runs; a pick saves at once and the
  picker then lives in Settings → Robot. Not shown with Jelly attached or
  on Mantis; the CLI still falls back to legacy.
- Settings saved elsewhere while the panel's draft is dirty no longer
  leave it stuck "unsaved": untouched keys follow the host, staged edits
  stay.

Co-Authored-By: Claude Opus 5.5 <noreply@anthropic.com>

File: almond_axol/kinematics/urdf/axol_jelly.urdf (robot description, URDF)
Before this commit: robot assembly, 43 links, 42 joints
Joints:
- joint floor_0: origin xyz=-0.112228 5.24549e-06 -0.46944 rpy=0 0 0 -> xyz=-0.112228 5.24549e-06 -0.469551 rpy=0 0 0

File: almond_axol/kinematics/urdf/axol_jelly_parcel.urdf (robot description, URDF)
Before this commit: robot assembly, 37 links, 36 joints
Joints:
- joint floor_0: origin xyz=-0.112228 5.36873e-06 -0.46944 rpy=0 0 0 -> xyz=-0.112228 5.36873e-06 -0.469551 rpy=0 0 0

File: almond_axol/kinematics/urdf/axol_ox_cart.urdf (robot description, URDF)
Before this commit: robot assembly, 35 links, 34 joints
Joints:
- joint floor_0: origin xyz=-0.100357 4.23699e-06 -0.31251 rpy=0 0 0 -> xyz=-0.100357 4.23699e-06 -0.425035 rpy=0 0 0
