Commit message: Ox cart: collide the lift's top plate on its own
The lift's top 38 mm is the plate the shoulder bar bolts onto, reaching
130 mm behind the 148 x 75 mm column. Folded into the column's IK hull it
widened pyroki's capsule to 127 mm and pulled it off the column toward
the back. It is now its own link (lift_plate, as on Jelly): the column
capsule is vertical at 108 mm and the plate a 122 mm disc on top.

Co-Authored-By: Claude Opus 5.5 <noreply@anthropic.com>

File: almond_axol/kinematics/urdf/axol_ox_cart.urdf (robot description, URDF)
Before this commit: robot assembly, 35 links, 34 joints
Links:
- added link lift_plate, mass 1; collision mesh filename=meshes/ox_cart/lift_plate_collision.stl scale=1 1 1
- link base: mass 6 -> 5; geometry collision mesh filename=meshes/ox_cart/base__column_top_collision.stl scale=1 1 1; visual mesh filename=meshes/ox_cart/base_0.stl scale=1 1 1
Joints:
- added joint lift_plate_0: type fixed, parent base, child lift_plate, origin xyz=0 0 0 rpy=0 0 0
